File: pkg/fan_controller/board/board.kicad_pcb (KiCad board)
At the start: 4 copper layers, 80 x 32 mm, 66 parts, among them J1 USB, J10 FAN3, J11 FAN4, J12 PUMP, J13 POWER_IN, J2 AVR-ISP-6, J3 FPANEL, J4 WATER_FLOW, J5 CPU, J6 WATER_TEMP, J7 AIR_TEMP, J8 FAN1, J9 FAN2, Q1 BSS138, Q2 BSS138, U1 ATmega32U4-MU, Y1 16MHz

Commit message: Flush changes.
Other:
- board text added: "CPU"
- board text added: "FAN1"
- board text added: "FAN2"
- board text added: "FAN3"
- board text added: "FAN4"
- board text added: "FLOW"
- board text added: "FPANEL"
- board text added: "PLED"
- board text added: "PUMP"
- board text added: "PWR+"
- board text added: "RST+"
- board text added: "TEMP1"
- board text added: "TEMP2"
- board text added: "USB"
Changed lines of the file:
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@@
   (general
     (thickness 1.6)
-    (drawings 10)
+    (drawings 36)
     (tracks 506)
     (zones 0)
@@
     (nets 68)
   )
-  (page A4)
+  (page USLetter)
   (layers
     (0 F.Cu signal)
@@
   )
   (setup
-    (last_trace_width 0.5)
+    (last_trace_width 0.25)
     (user_trace_width 0.5)
     (trace_clearance 0.2)
@@
     )
   )
-  (module Diode_SMD:D_0603_1608Metric (layer F.Cu)
+  (module Diode_SMD:D_0603_1608Metric locked (layer F.Cu)
     (at 118 62.5 90)
     (descr "Diode SMD 0603 (1608 Metric), square (rectangular) end terminal, IPC_7351 nominal, (Body size source: http://www.tortai-tech.com/upload/download/2011102023233369053.pdf), generated with kicad-footprint-generator")
@@
     )
   )
+  (gr_line (start 151.13 80.264) (end 150.876 77.978) (layer Dwgs.User) (width 0.15))
+  (gr_line (start 154.94 80.264) (end 151.13 80.264) (layer Dwgs.User) (width 0.15))
+  (gr_line (start 154.94 77.978) (end 154.94 80.264) (layer Dwgs.User) (width 0.15))
+  (gr_line (start 150.876 77.978) (end 154.94 77.978) (layer Dwgs.User) (width 0.15))
+  (gr_line (start 116.586 64.262) (end 116.84 60.452) (layer Dwgs.User) (width 0.15))
+  (gr_line (start 129.794 64.262) (end 116.586 64.262) (layer Dwgs.User) (width 0.15))
+  (gr_line (start 129.54 60.452) (end 129.794 64.262) (layer Dwgs.User) (width 0.15))
+  (gr_line (start 116.84 60.452) (end 129.54 60.452) (layer Dwgs.User) (width 0.15))
+  (gr_text PUMP (at 174.498 47.498) (layer Dwgs.User)
+    (effects (font (size 1.5 1.5) (thickness 0.3)))
+  )
+  (gr_text CPU (at 161.798 47.244) (layer Dwgs.User)
+    (effects (font (size 1.5 1.5) (thickness 0.3)))
+  )
+  (gr_text FAN4 (at 149.352 47.498) (layer Dwgs.User)
+    (effects (font (size 1.5 1.5) (thickness 0.3)))
+  )
+  (gr_text FAN3 (at 136.652 47.498) (layer Dwgs.User)
+    (effects (font (size 1.5 1.5) (thickness 0.3)))
+  )
+  (gr_text FAN2 (at 123.698 47.498) (layer Dwgs.User)
+    (effects (font (size 1.5 1.5) (thickness 0.3)))
+  )
+  (gr_text FAN1 (at 110.998 47.498) (layer Dwgs.User)
+    (effects (font (size 1.5 1.5) (thickness 0.3)))
+  )
+  (gr_text TEMP2 (at 105.918 63.246) (layer Dwgs.User)
+    (effects (font (size 1.5 1.5) (thickness 0.3)))
+  )
+  (gr_text TEMP1 (at 105.918 70.866) (layer Dwgs.User)
+    (effects (font (size 1.5 1.5) (thickness 0.3)))
+  )
+  (gr_text FLOW (at 105.156 78.486) (layer Dwgs.User)
+    (effects (font (size 1.5 1.5) (thickness 0.3)))
+  )
+  (gr_text USB (at 169.672 75.438 90) (layer Dwgs.User)
+    (effects (font (size 1.5 1.5) (thickness 0.3)))
+  )
+  (gr_text FPANEL (at 169.672 64.262 90) (layer Dwgs.User)
+    (effects (font (size 1.5 1.5) (thickness 0.3)))
+  )
+  (gr_text RST+ (at 175.514 66.802) (layer Dwgs.User)
+    (effects (font (size 1.5 1.5) (thickness 0.3)))
+  )
+  (gr_text PWR+ (at 175.768 64.262) (layer Dwgs.User)
+    (effects (font (size 1.5 1.5) (thickness 0.3)))
+  )
+  (gr_text PLED (at 175.26 61.722) (layer Dwgs.User)
+    (effects (font (size 1.5 1.5) (thickness 0.3)))
+  )
+  (gr_text GND (at 175.006 79.502) (layer Dwgs.User)
+    (effects (font (size 1.5 1.5) (thickness 0.3)))
+  )
+  (gr_text D- (at 174.498 76.962) (layer Dwgs.User)
+    (effects (font (size 1.5 1.5) (thickness 0.3)))
+  )
+  (gr_text D+ (at 174.498 74.422) (layer Dwgs.User)
+    (effects (font (size 1.5 1.5) (thickness 0.3)))
+  )
+  (gr_text +5V (at 174.752 71.374) (layer Dwgs.User)
+    (effects (font (size 1.5 1.5) (thickness 0.3)))
+  )
   (gr_text GND (at 173.4312 79.4512) (layer F.SilkS)
