File: pkg/fan_controller/board/board.sch (KiCad schematic (older format))
At the start: 66 parts, among them J1 USB, J10 FAN3, J11 FAN4, J12 PUMP, J13 POWER_IN, J2 AVR-ISP-6, J3 FPANEL, J4 WATER_FLOW, J5 CPU, J6 WATER_TEMP, J7 AIR_TEMP, J8 FAN1, J9 FAN2, Q1 BSS138, Q2 BSS138, U1 ATmega32U4-MU, Y1 16MHz

Commit message: Flush misc changes.
Parts:
- removed C1, C2: 22pF, Capacitor_SMD:C_0603_1608Metric, symbol Device:C_Small
- removed C3: 0.1uF, Capacitor_SMD:C_0603_1608Metric, symbol Device:C_Small
- removed C4, C5: 1uF, Capacitor_SMD:C_0603_1608Metric, symbol Device:C_Small
- removed C6, C7, C8, C9: 10uF, Capacitor_SMD:C_0805_2012Metric, symbol Device:C_Small
- removed D1, D2, D3, D4, D5, D6: BLUE, Diode_SMD:D_0603_1608Metric, symbol Device:LED
- removed F1: 100mA, Fuse:Fuse_0603_1608Metric, symbol Device:Polyfuse_Small
- removed J1: USB, Connector_PinHeader_2.54mm:PinHeader_1x04_P2.54mm_Horizontal, symbol Connector:Conn_01x04_Male
- removed J10: FAN3, Connector_PinHeader_2.54mm:PinHeader_1x04_P2.54mm_Horizontal, symbol Connector:Conn_01x04_Male
- removed J11: FAN4, Connector_PinHeader_2.54mm:PinHeader_1x04_P2.54mm_Horizontal, symbol Connector:Conn_01x04_Male
- removed J12: PUMP, Connector_PinHeader_2.54mm:PinHeader_1x04_P2.54mm_Horizontal, symbol Connector:Conn_01x04_Male
- removed J13: POWER_IN, Connector_PinHeader_2.54mm:PinHeader_1x02_P2.54mm_Vertical, symbol Connector:Conn_01x02_Male
- removed J2: AVR-ISP-6, Connector_PinHeader_2.54mm:PinHeader_2x03_P2.54mm_Vertical, symbol Connector:AVR-ISP-6
- removed J3: FPANEL, Connector_PinHeader_2.54mm:PinHeader_1x03_P2.54mm_Horizontal, symbol Connector:Conn_01x03_Male
- removed J4: WATER_FLOW, Connector_PinHeader_2.54mm:PinHeader_1x02_P2.54mm_Horizontal, symbol Connector:Conn_01x02_Male
- removed J5: CPU, Connector_PinHeader_2.54mm:PinHeader_1x04_P2.54mm_Horizontal, symbol Connector:Conn_01x04_Male
- removed J6: WATER_TEMP, Connector_PinHeader_2.54mm:PinHeader_1x02_P2.54mm_Horizontal, symbol Connector:Conn_01x02_Male
- removed J7: AIR_TEMP, Connector_PinHeader_2.54mm:PinHeader_1x02_P2.54mm_Horizontal, symbol Connector:Conn_01x02_Male
- removed J8: FAN1, Connector_PinHeader_2.54mm:PinHeader_1x04_P2.54mm_Horizontal, symbol Connector:Conn_01x04_Male
- removed J9: FAN2, Connector_PinHeader_2.54mm:PinHeader_1x04_P2.54mm_Horizontal, symbol Connector:Conn_01x04_Male
- removed Q1, Q2: BSS138, Package_TO_SOT_SMD:SOT-23, symbol Transistor_FET:BSS138
- removed R10, R8: 1K, Resistor_SMD:R_0603_1608Metric, symbol Device:R_Small
- removed R11, R15, R16, R17, R18, R19, R20, R21, R22, R23, R24, R25, R26, R27, R28, R30, R7, R9: 500, Resistor_SMD:R_0603_1608Metric, symbol Device:R_Small
- removed R12, R29, R3: 10K, Resistor_SMD:R_0603_1608Metric, symbol Device:R_Small
- removed R13, R14: 5.6K, Resistor_SMD:R_0603_1608Metric, symbol Device:R_Small
- removed R2: 22, Resistor_SMD:R_0603_1608Metric, symbol Device:R_Small
- removed R31, R32, R33, R4, R5, R6: 330, Resistor_SMD:R_0603_1608Metric, symbol Device:R_Small
- removed U1: ATmega32U4-MU, Package_DFN_QFN:QFN-44-1EP_7x7mm_P0.5mm_EP5.2x5.2mm, symbol MCU_Microchip_ATmega:ATmega32U4-MU
- removed Y1: 16MHz, Crystal:Crystal_SMD_3225-4Pin_3.2x2.5mm, symbol Device:Crystal_GND24_Small
- added A1: TINY2040, tiny2040:tiny2040, symbol tiny2040:TINY2040
- added C?: 10uF, symbol Device:C_Small
- added C?: 10nF, symbol Device:C_Small
- added J1: Conn_01x04, symbol Connector_Generic:Conn_01x04
- added J? (x3): Conn_01x02, symbol Connector_Generic:Conn_01x02
- added Q?: 2N7000, Package_TO_SOT_THT:TO-92_Inline, symbol Transistor_FET:2N7000
- added R? (x5): 500, symbol Device:R_Small
- added R?: 5.6K, symbol Device:R_Small
- added U?: LM1117-3.3, symbol Regulator_Linear:LM1117-3.3
- R1: value 22 -> 500; footprint Resistor_SMD:R_0603_1608Metric -> (none); LCSC C23345 -> (none)
Connections:
- net FAN_PWM_A: now also A1.0, Q?.2 (G)
- net FAN_PWM_B: now also A1.1
- net FAN_PWM_C: now also A1.2
- net FAN_SPEED_1: now also R1.2, A1.3
- net FAN_SPEED_2: now also A1.4
- net FAN_SPEED_3: now also A1.5
- net FAN_SPEED_4: now also A1.6
- net FAN_SPEED_5: now also A1.7
- net GND: now also A1.GND1, A1.GND2, A1.GND3, C?.2, C?.2, J1.4 (Pin_4), J?.2 (Pin_2), Q?.1 (S), R?.1, R?.2, U?.1 (GND)
- net D+: no longer names the net of R1.1
- net D+: now also J1.2 (Pin_2)
- new net: J1.1 (Pin_1), R?.1
- new net: Q?.3 (D), R?.2
- new net: J?.2 (Pin_2), R?.2 (x2)
- new net: J?.1 (Pin_1), R?.1
- new net +12V: C?.1, J1.3 (Pin_3), J?.1 (Pin_1), U?.3 (VI)
- new net +3V3: A1.3V3, C?.1, R?.1, U?.2 (VO)
- new net FLOW_CH1: A1.A3, R?.2
- new net TEMP_CH1: A1.A1, R?.1, R?.1
- new net TEMP_CH2: A1.A0
- new net TEMP_VDD: J?.1 (Pin_1), R?.2
Other:
- note added: "FANX_PWM pulled-down in MCU.\nFANX_SPEED pulled-up in MCU."
- note added: "WATER_FLOW should be pulled-up in the MCU"
