File: doc/keyboard/board/board.kicad_pcb (KiCad board)
At the start: 4 copper layers, 363 x 128 mm, 302 parts, among them J1 OLED, J2 Conn_01x05, J3 Conn_01x03, J4 Conn_02x03_Odd_Even, Q1 DMG2305, Q2 DM2305, Q3 2N7002, SW1 SW_Push, SW10 SW_Push, SW11 SW_Push, SW12 SW_Push, SW13 SW_Push, SW14 SW_Push, SW15 SW_Push, SW16 SW_Push, SW17 SW_Push, SW18 SW_Push, SW19 SW_Push, SW2 SW_Push, SW20 SW_Push, SW21 SW_Push, SW22 SW_Push, SW23 SW_Push, SW24 SW_Push, SW25 SW_Push, SW26 SW_Push, SW27 SW_Push, SW28 SW_Push, SW29 SW_Push, SW3 SW_Push, SW30 SW_Push, SW31 SW_Push, SW32 SW_Push, SW33 SW_Push, SW34 SW_Push, SW35 SW_Push, SW36 SW_Push, SW37 SW_Push, SW38 SW_Push, SW39 SW_Push, SW4 SW_Push, SW40 SW_Push, SW41 SW_Push, SW42 SW_Push, SW43 SW_Push, SW44 SW_Push, SW45 SW_Push, SW46 SW_Push, SW47 SW_Push, SW48 SW_Push, SW49 SW_Push, SW5 SW_Push, SW50 SW_Push, SW51 SW_Push, SW52 SW_Push, SW53 SW_Push, SW54 SW_Push, SW55 SW_Push, SW56 SW_Push, SW57 SW_Push, SW58 SW_Push, SW59 SW_Push, SW6 SW_Push, SW60 SW_Push, SW61 SW_Push, SW62 SW_Push, SW63 SW_Push, SW64 SW_Push, SW65 SW_Push, SW66 SW_Push, SW67 SW_Push, SW68 SW_Push, SW69 SW_Push, SW7 SW_Push, SW70 SW_Push, SW71 SW_Push, SW72 SW_Push, SW73 SW_Push, SW74 SW_Push, SW75 SW_Push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

Commit message: Keyboard with all LED caps placed.
Parts:
- added CS1: 0.1uF, Capacitor_SMD:C_0805_2012Metric_Pad1.15x1.40mm_HandSolder, B.Cu at (112.6, 121.8)
- added CS10: 0.1uF, Capacitor_SMD:C_0805_2012Metric_Pad1.15x1.40mm_HandSolder, B.Cu at (333.8, 117.0)
- added CS11: 0.1uF, Capacitor_SMD:C_0805_2012Metric_Pad1.15x1.40mm_HandSolder, B.Cu at (352.9, 117.0)
- added CS12: 0.1uF, Capacitor_SMD:C_0805_2012Metric_Pad1.15x1.40mm_HandSolder, B.Cu at (371.9, 117.0)
- added CS13: 0.1uF, Capacitor_SMD:C_0805_2012Metric_Pad1.15x1.40mm_HandSolder, B.Cu at (391.0, 117.0)
- added CS14: 0.1uF, Capacitor_SMD:C_0805_2012Metric_Pad1.15x1.40mm_HandSolder, B.Cu at (414.8, 117.0)
- added CS15: 0.1uF, Capacitor_SMD:C_0805_2012Metric_Pad1.15x1.40mm_HandSolder, B.Cu at (433.9, 117.0)
- added CS16: 0.1uF, Capacitor_SMD:C_0805_2012Metric_Pad1.15x1.40mm_HandSolder, B.Cu at (452.9, 117.0)
- added CS17: 0.1uF, Capacitor_SMD:C_0805_2012Metric_Pad1.15x1.40mm_HandSolder, B.Cu at (452.9, 145.5)
- added CS18: 0.1uF, Capacitor_SMD:C_0805_2012Metric_Pad1.15x1.40mm_HandSolder, B.Cu at (433.9, 145.5)
- added CS19: 0.1uF, Capacitor_SMD:C_0805_2012Metric_Pad1.15x1.40mm_HandSolder, B.Cu at (414.8, 145.5)
- added CS2: 0.1uF, Capacitor_SMD:C_0805_2012Metric_Pad1.15x1.40mm_HandSolder, B.Cu at (162.4, 117.0)
- added CS20: 0.1uF, Capacitor_SMD:C_0805_2012Metric_Pad1.15x1.40mm_HandSolder, B.Cu at (381.5, 145.5)
- added CS21: 0.1uF, Capacitor_SMD:C_0805_2012Metric_Pad1.15x1.40mm_HandSolder, B.Cu at (352.9, 145.5)
- added CS22: 0.1uF, Capacitor_SMD:C_0805_2012Metric_Pad1.15x1.40mm_HandSolder, B.Cu at (333.8, 145.5)
- added CS23: 0.1uF, Capacitor_SMD:C_0805_2012Metric_Pad1.15x1.40mm_HandSolder, B.Cu at (314.8, 145.5)
- added CS24: 0.1uF, Capacitor_SMD:C_0805_2012Metric_Pad1.15x1.40mm_HandSolder, B.Cu at (295.7, 145.5)
- added CS25: 0.1uF, Capacitor_SMD:C_0805_2012Metric_Pad1.15x1.40mm_HandSolder, B.Cu at (276.7, 145.5)
- added CS26: 0.1uF, Capacitor_SMD:C_0805_2012Metric_Pad1.15x1.40mm_HandSolder, B.Cu at (257.6, 145.5)
- added CS27: 0.1uF, Capacitor_SMD:C_0805_2012Metric_Pad1.15x1.40mm_HandSolder, B.Cu at (238.6, 145.5)
- added CS28: 0.1uF, Capacitor_SMD:C_0805_2012Metric_Pad1.15x1.40mm_HandSolder, B.Cu at (219.5, 145.5)
- added CS29: 0.1uF, Capacitor_SMD:C_0805_2012Metric_Pad1.15x1.40mm_HandSolder, B.Cu at (200.5, 145.5)
- added CS3: 0.1uF, Capacitor_SMD:C_0805_2012Metric_Pad1.15x1.40mm_HandSolder, B.Cu at (181.4, 117.0)
- added CS30: 0.1uF, Capacitor_SMD:C_0805_2012Metric_Pad1.15x1.40mm_HandSolder, B.Cu at (181.4, 145.5)
- added CS31: 0.1uF, Capacitor_SMD:C_0805_2012Metric_Pad1.15x1.40mm_HandSolder, B.Cu at (162.4, 145.5)
- added CS32: 0.1uF, Capacitor_SMD:C_0805_2012Metric_Pad1.15x1.40mm_HandSolder, B.Cu at (143.3, 145.5)
- added CS33: 0.1uF, Capacitor_SMD:C_0805_2012Metric_Pad1.15x1.40mm_HandSolder, B.Cu at (124.3, 145.5)
- added CS34: 0.1uF, Capacitor_SMD:C_0805_2012Metric_Pad1.15x1.40mm_HandSolder, B.Cu at (129.1, 164.6)
- added CS35: 0.1uF, Capacitor_SMD:C_0805_2012Metric_Pad1.15x1.40mm_HandSolder, B.Cu at (152.9, 164.6)
- added CS36: 0.1uF, Capacitor_SMD:C_0805_2012Metric_Pad1.15x1.40mm_HandSolder, B.Cu at (171.9, 164.6)
- added CS37: 0.1uF, Capacitor_SMD:C_0805_2012Metric_Pad1.15x1.40mm_HandSolder, B.Cu at (191.0, 164.6)
- added CS38: 0.1uF, Capacitor_SMD:C_0805_2012Metric_Pad1.15x1.40mm_HandSolder, B.Cu at (210.0, 164.6)
- added CS39: 0.1uF, Capacitor_SMD:C_0805_2012Metric_Pad1.15x1.40mm_HandSolder, B.Cu at (229.1, 164.6)
- added CS4: 0.1uF, Capacitor_SMD:C_0805_2012Metric_Pad1.15x1.40mm_HandSolder, B.Cu at (200.5, 117.0)
- added CS40: 0.1uF, Capacitor_SMD:C_0805_2012Metric_Pad1.15x1.40mm_HandSolder, B.Cu at (248.1, 164.6)
- added CS41: 0.1uF, Capacitor_SMD:C_0805_2012Metric_Pad1.15x1.40mm_HandSolder, B.Cu at (267.2, 164.6)
- added CS42: 0.1uF, Capacitor_SMD:C_0805_2012Metric_Pad1.15x1.40mm_HandSolder, B.Cu at (286.2, 164.6)
- added CS43: 0.1uF, Capacitor_SMD:C_0805_2012Metric_Pad1.15x1.40mm_HandSolder, B.Cu at (305.3, 164.6)
- added CS44: 0.1uF, Capacitor_SMD:C_0805_2012Metric_Pad1.15x1.40mm_HandSolder, B.Cu at (324.3, 164.6)
- added CS45: 0.1uF, Capacitor_SMD:C_0805_2012Metric_Pad1.15x1.40mm_HandSolder, B.Cu at (343.4, 164.6)
- added CS46: 0.1uF, Capacitor_SMD:C_0805_2012Metric_Pad1.15x1.40mm_HandSolder, B.Cu at (362.4, 164.6)
- added CS47: 0.1uF, Capacitor_SMD:C_0805_2012Metric_Pad1.15x1.40mm_HandSolder, B.Cu at (386.2, 164.6)
- added CS48: 0.1uF, Capacitor_SMD:C_0805_2012Metric_Pad1.15x1.40mm_HandSolder, B.Cu at (414.8, 164.6)
- added CS49: 0.1uF, Capacitor_SMD:C_0805_2012Metric_Pad1.15x1.40mm_HandSolder, B.Cu at (433.9, 164.6)
- added CS5: 0.1uF, Capacitor_SMD:C_0805_2012Metric_Pad1.15x1.40mm_HandSolder, B.Cu at (218.4, 116.8)
- added CS50: 0.1uF, Capacitor_SMD:C_0805_2012Metric_Pad1.15x1.40mm_HandSolder, B.Cu at (452.9, 164.6)
- added CS51: 0.1uF, Capacitor_SMD:C_0805_2012Metric_Pad1.15x1.40mm_HandSolder, B.Cu at (379.1, 183.6)
- added CS52: 0.1uF, Capacitor_SMD:C_0805_2012Metric_Pad1.15x1.40mm_HandSolder, B.Cu at (348.1, 183.6)
- added CS53: 0.1uF, Capacitor_SMD:C_0805_2012Metric_Pad1.15x1.40mm_HandSolder, B.Cu at (329.1, 183.6)
- added CS54: 0.1uF, Capacitor_SMD:C_0805_2012Metric_Pad1.15x1.40mm_HandSolder, B.Cu at (310.0, 183.6)
- added CS55: 0.1uF, Capacitor_SMD:C_0805_2012Metric_Pad1.15x1.40mm_HandSolder, B.Cu at (291.0, 183.6)
- added CS56: 0.1uF, Capacitor_SMD:C_0805_2012Metric_Pad1.15x1.40mm_HandSolder, B.Cu at (271.9, 183.6)
- added CS57: 0.1uF, Capacitor_SMD:C_0805_2012Metric_Pad1.15x1.40mm_HandSolder, B.Cu at (252.9, 183.6)
- added CS58: 0.1uF, Capacitor_SMD:C_0805_2012Metric_Pad1.15x1.40mm_HandSolder, B.Cu at (233.8, 183.6)
- added CS59: 0.1uF, Capacitor_SMD:C_0805_2012Metric_Pad1.15x1.40mm_HandSolder, B.Cu at (214.8, 183.6)
- added CS6: 0.1uF, Capacitor_SMD:C_0805_2012Metric_Pad1.15x1.40mm_HandSolder, B.Cu at (248.1, 117.0)
- added CS60: 0.1uF, Capacitor_SMD:C_0805_2012Metric_Pad1.15x1.40mm_HandSolder, B.Cu at (195.7, 183.6)
- added CS61: 0.1uF, Capacitor_SMD:C_0805_2012Metric_Pad1.15x1.40mm_HandSolder, B.Cu at (176.7, 183.6)
- added CS62: 0.1uF, Capacitor_SMD:C_0805_2012Metric_Pad1.15x1.40mm_HandSolder, B.Cu at (157.6, 183.6)
- added CS63: 0.1uF, Capacitor_SMD:C_0805_2012Metric_Pad1.15x1.40mm_HandSolder, B.Cu at (131.4, 183.6)
- added CS64: 0.1uF, Capacitor_SMD:C_0805_2012Metric_Pad1.15x1.40mm_HandSolder, B.Cu at (136.2, 202.7)
- added CS65: 0.1uF, Capacitor_SMD:C_0805_2012Metric_Pad1.15x1.40mm_HandSolder, B.Cu at (167.2, 202.7)
- added CS66: 0.1uF, Capacitor_SMD:C_0805_2012Metric_Pad1.15x1.40mm_HandSolder, B.Cu at (186.2, 202.7)
- added CS67: 0.1uF, Capacitor_SMD:C_0805_2012Metric_Pad1.15x1.40mm_HandSolder, B.Cu at (205.3, 202.7)
- added CS68: 0.1uF, Capacitor_SMD:C_0805_2012Metric_Pad1.15x1.40mm_HandSolder, B.Cu at (224.3, 202.7)
- added CS69: 0.1uF, Capacitor_SMD:C_0805_2012Metric_Pad1.15x1.40mm_HandSolder, B.Cu at (243.4, 202.7)
- added CS7: 0.1uF, Capacitor_SMD:C_0805_2012Metric_Pad1.15x1.40mm_HandSolder, B.Cu at (267.2, 117.0)
- added CS70: 0.1uF, Capacitor_SMD:C_0805_2012Metric_Pad1.15x1.40mm_HandSolder, B.Cu at (262.4, 202.7)
- added CS71: 0.1uF, Capacitor_SMD:C_0805_2012Metric_Pad1.15x1.40mm_HandSolder, B.Cu at (281.5, 202.7)
- added CS72: 0.1uF, Capacitor_SMD:C_0805_2012Metric_Pad1.15x1.40mm_HandSolder, B.Cu at (300.5, 202.7)
- added CS73: 0.1uF, Capacitor_SMD:C_0805_2012Metric_Pad1.15x1.40mm_HandSolder, B.Cu at (319.6, 202.7)
- added CS74: 0.1uF, Capacitor_SMD:C_0805_2012Metric_Pad1.15x1.40mm_HandSolder, B.Cu at (338.6, 202.7)
- added CS75: 0.1uF, Capacitor_SMD:C_0805_2012Metric_Pad1.15x1.40mm_HandSolder, B.Cu at (374.3, 202.7)
- added CS76: 0.1uF, Capacitor_SMD:C_0805_2012Metric_Pad1.15x1.40mm_HandSolder, B.Cu at (433.9, 202.7)
- added CS77: 0.1uF, Capacitor_SMD:C_0805_2012Metric_Pad1.15x1.40mm_HandSolder, B.Cu at (452.9, 221.7)
- added CS78: 0.1uF, Capacitor_SMD:C_0805_2012Metric_Pad1.15x1.40mm_HandSolder, B.Cu at (433.9, 221.7)
- added CS79: 0.1uF, Capacitor_SMD:C_0805_2012Metric_Pad1.15x1.40mm_HandSolder, B.Cu at (414.8, 221.7)
- added CS8: 0.1uF, Capacitor_SMD:C_0805_2012Metric_Pad1.15x1.40mm_HandSolder, B.Cu at (286.2, 117.0)
- added CS80: 0.1uF, Capacitor_SMD:C_0805_2012Metric_Pad1.15x1.40mm_HandSolder, B.Cu at (388.6, 221.7)
- added CS81: 0.1uF, Capacitor_SMD:C_0805_2012Metric_Pad1.15x1.40mm_HandSolder, B.Cu at (364.8, 221.7)
- added CS82: 0.1uF, Capacitor_SMD:C_0805_2012Metric_Pad1.15x1.40mm_HandSolder, B.Cu at (341.0, 221.7)
- added CS83: 0.1uF, Capacitor_SMD:C_0805_2012Metric_Pad1.15x1.40mm_HandSolder, B.Cu at (317.2, 221.7)
- added CS84: 0.1uF, Capacitor_SMD:C_0805_2012Metric_Pad1.15x1.40mm_HandSolder, B.Cu at (245.7, 221.7)
- added CS85: 0.1uF, Capacitor_SMD:C_0805_2012Metric_Pad1.15x1.40mm_HandSolder, B.Cu at (174.3, 221.7)
- added CS86: 0.1uF, Capacitor_SMD:C_0805_2012Metric_Pad1.15x1.40mm_HandSolder, B.Cu at (150.5, 221.7)
- added CS87: 0.1uF, Capacitor_SMD:C_0805_2012Metric_Pad1.15x1.40mm_HandSolder, B.Cu at (126.7, 221.7)
- added CS9: 0.1uF, Capacitor_SMD:C_0805_2012Metric_Pad1.15x1.40mm_HandSolder, B.Cu at (305.3, 117.0)
- moved J1 2.64 mm to (401.0, 179.3)
Routing:
- net LED_GND: track 237.4 -> 388.9 mm, vias 102 -> 147
- net LED_VDD: track 190.5 -> 340.7 mm, vias 89 -> 130
- net KEY_Y4: track 528.2 -> 524.1 mm
- net KEY_X_REGISTER_CLEAR: track 299.3 -> 303.1 mm
- net Net-(E50-Pad2): track 89.2 -> 93.0 mm
- net Net-(E16-Pad2): track 36.0 -> 39.2 mm
- net CHARGE_STAT: track 110.3 -> 112.4 mm
- net Net-(U3-Pad9): track 174.2 -> 175.7 mm
- net KEY_X_REGISTER_CLK: track 185.6 -> 184.4 mm
- net SCL: track 362.7 -> 363.9 mm
- net SDA: track 365.2 -> 366.4 mm

Commit message: More keyboard documentation and polishing.
Parts:
- added CS100: 0.1uF, Capacitor_SMD:C_0603_1608Metric_Pad1.05x0.95mm_HandSolder, B.Cu at (458.0, 160.0)
- added CS101: 0.1uF, Capacitor_SMD:C_0603_1608Metric_Pad1.05x0.95mm_HandSolder, B.Cu at (458.0, 150.0)
- added CS102: 0.1uF, Capacitor_SMD:C_0603_1608Metric_Pad1.05x0.95mm_HandSolder, B.Cu at (458.0, 140.0)
- added CS103: 0.1uF, Capacitor_SMD:C_0603_1608Metric_Pad1.05x0.95mm_HandSolder, B.Cu at (458.0, 130.0)
- added CS88: 0.1uF, Capacitor_SMD:C_0603_1608Metric_Pad1.05x0.95mm_HandSolder, B.Cu at (107.0, 200.0)
- added CS89: 0.1uF, Capacitor_SMD:C_0603_1608Metric_Pad1.05x0.95mm_HandSolder, B.Cu at (107.0, 190.0)
- added CS90: 0.1uF, Capacitor_SMD:C_0603_1608Metric_Pad1.05x0.95mm_HandSolder, B.Cu at (107.0, 180.0)
- added CS91: 0.1uF, Capacitor_SMD:C_0603_1608Metric_Pad1.05x0.95mm_HandSolder, B.Cu at (107.0, 170.0)
- added CS92: 0.1uF, Capacitor_SMD:C_0603_1608Metric_Pad1.05x0.95mm_HandSolder, B.Cu at (107.0, 160.0)
- added CS93: 0.1uF, Capacitor_SMD:C_0603_1608Metric_Pad1.05x0.95mm_HandSolder, B.Cu at (107.0, 150.0)
- added CS94: 0.1uF, Capacitor_SMD:C_0603_1608Metric_Pad1.05x0.95mm_HandSolder, B.Cu at (107.0, 140.0)
- added CS95: 0.1uF, Capacitor_SMD:C_0603_1608Metric_Pad1.05x0.95mm_HandSolder, B.Cu at (107.0, 130.0)
- added CS96: 0.1uF, Capacitor_SMD:C_0603_1608Metric_Pad1.05x0.95mm_HandSolder, B.Cu at (458.0, 200.0)
- added CS97: 0.1uF, Capacitor_SMD:C_0603_1608Metric_Pad1.05x0.95mm_HandSolder, B.Cu at (458.0, 190.0)
- added CS98: 0.1uF, Capacitor_SMD:C_0603_1608Metric_Pad1.05x0.95mm_HandSolder, B.Cu at (458.0, 180.0)
- added CS99: 0.1uF, Capacitor_SMD:C_0603_1608Metric_Pad1.05x0.95mm_HandSolder, B.Cu at (458.0, 170.0)
- added E100: SK6812MINI-E, Components:SK6812B-SIDE, B.Cu at (459.0, 160.0)
- added E101: SK6812MINI-E, Components:SK6812B-SIDE, B.Cu at (459.0, 150.0)
- added E102: SK6812MINI-E, Components:SK6812B-SIDE, B.Cu at (459.0, 140.0)
- added E103: SK6812MINI-E, Components:SK6812B-SIDE, B.Cu at (459.0, 130.0)
- added E88: SK6812MINI-E, Components:SK6812B-SIDE, B.Cu at (106.0, 200.0)
- added E89: SK6812MINI-E, Components:SK6812B-SIDE, B.Cu at (106.0, 190.0)
- added E90: SK6812MINI-E, Components:SK6812B-SIDE, B.Cu at (106.0, 180.0)
- added E91: SK6812MINI-E, Components:SK6812B-SIDE, B.Cu at (106.0, 170.0)
- added E92: SK6812MINI-E, Components:SK6812B-SIDE, B.Cu at (106.0, 160.0)
- added E93: SK6812MINI-E, Components:SK6812B-SIDE, B.Cu at (106.0, 150.0)
- added E94: SK6812MINI-E, Components:SK6812B-SIDE, B.Cu at (106.0, 140.0)
- added E95: SK6812MINI-E, Components:SK6812B-SIDE, B.Cu at (106.0, 130.0)
- added E96: SK6812MINI-E, Components:SK6812B-SIDE, B.Cu at (459.0, 200.0)
- added E97: SK6812MINI-E, Components:SK6812B-SIDE, B.Cu at (459.0, 190.0)
- added E98: SK6812MINI-E, Components:SK6812B-SIDE, B.Cu at (459.0, 180.0)
- added E99: SK6812MINI-E, Components:SK6812B-SIDE, B.Cu at (459.0, 170.0)
- added FID1: Fiducial, Fiducial:Fiducial_1mm_Mask2mm, B.Cu at (435.3, 126.8)
- added FID2: Fiducial, Fiducial:Fiducial_1mm_Mask2mm, B.Cu at (134.3, 160.1)
- added FID3: Fiducial, Fiducial:Fiducial_1mm_Mask2mm, B.Cu at (104.9, 224.7)
- added FID4: Fiducial, Fiducial:Fiducial_1mm_Mask2mm, B.Cu at (104.7, 105.9)
- added FID5: Fiducial, Fiducial:Fiducial_1mm_Mask2mm, B.Cu at (258.3, 216.9)
- added FID6: Fiducial, Fiducial:Fiducial_1mm_Mask2mm, B.Cu at (313.4, 111.1)
- added FID7: Fiducial, Fiducial:Fiducial_1mm_Mask2mm, B.Cu at (460.1, 105.6)
- added FID8: Fiducial, Fiducial:Fiducial_1mm_Mask2mm, B.Cu at (460.4, 224.4)
- added J5: Conn_01x02, Connector_PinHeader_2.54mm:PinHeader_1x02_P2.54mm_Vertical, B.Cu at (141.6, 126.3)
- Q2: value DM2305 -> DMG2305
- SW63: moved to F.Cu
- turned SW63 to 90 degrees
Connections:
- E87 pad 2: Net-(E87-Pad2) -> LED_SERIAL_8
- SW63 pad 1: Net-(D63-Pad2) -> KEY_X15
- SW63 pad 2: KEY_X15 -> Net-(D63-Pad2)
Routing:
- net Net-(E95-Pad2): track 0.00 -> 479.7 mm, vias 0 -> 2
- net LED_GND: track 388.9 -> 449.6 mm, vias 147 -> 163
- net LED_VDD: track 340.7 -> 400.7 mm, vias 130 -> 146
- net LED_SERIAL_8: track 0.00 -> 28.5 mm
- net Net-(E100-Pad4): track 0.00 -> 16.1 mm
- net Net-(E98-Pad2): track 0.00 -> 15.9 mm
- net Net-(E97-Pad2): track 0.00 -> 15.9 mm
- net Net-(E96-Pad2): track 0.00 -> 15.9 mm
- net Net-(E102-Pad2): track 0.00 -> 15.9 mm
- net Net-(E101-Pad2): track 0.00 -> 15.9 mm
- net Net-(E100-Pad2): track 0.00 -> 15.9 mm
- net Net-(E91-Pad2): track 0.00 -> 11.9 mm
- net Net-(E93-Pad2): track 0.00 -> 9.13 mm
- net Net-(E94-Pad2): track 0.00 -> 8.99 mm
- net Net-(E92-Pad2): track 0.00 -> 8.99 mm
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