File: doc/keyboard/board/board.sch (KiCad schematic (older format))
At the start: 303 parts, among them J1 OLED, J2 Conn_01x05, J3 Conn_01x03, J4 Conn_02x03_Odd_Even, Q1 DMG2305, Q2 DM2305, Q3 2N7002, SW1 SW_Push, SW10 SW_Push, SW11 SW_Push, SW12 SW_Push, SW13 SW_Push, SW14 SW_Push, SW15 SW_Push, SW16 SW_Push, SW17 SW_Push, SW18 SW_Push, SW19 SW_Push, SW2 SW_Push, SW20 SW_Push, SW21 SW_Push, SW22 SW_Push, SW23 SW_Push, SW24 SW_Push, SW25 SW_Push, SW26 SW_Push, SW27 SW_Push, SW28 SW_Push, SW29 SW_Push, SW3 SW_Push, SW30 SW_Push, SW31 SW_Push, SW32 SW_Push, SW33 SW_Push, SW34 SW_Push, SW35 SW_Push, SW36 SW_Push, SW37 SW_Push, SW38 SW_Push, SW39 SW_Push, SW4 SW_Push, SW40 SW_Push, SW41 SW_Push, SW42 SW_Push, SW43 SW_Push, SW44 SW_Push, SW45 SW_Push, SW46 SW_Push, SW47 SW_Push, SW48 SW_Push, SW49 SW_Push, SW5 SW_Push, SW50 SW_Push, SW51 SW_Push, SW52 SW_Push, SW53 SW_Push, SW54 SW_Push, SW55 SW_Push, SW56 SW_Push, SW57 SW_Push, SW58 SW_Push, SW59 SW_Push, SW6 SW_Push, SW60 SW_Push, SW61 SW_Push, SW62 SW_Push, SW63 SW_Push, SW64 SW_Push, SW65 SW_Push, SW66 SW_Push, SW67 SW_Push, SW68 SW_Push, SW69 SW_Push, SW7 SW_Push, SW70 SW_Push, SW71 SW_Push, SW72 SW_Push, SW73 SW_Push, SW74 SW_Push, SW75 SW_Push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

Commit message: Keyboard with all LED caps placed.
Parts:
- added CS10, CS11, CS12, CS13, CS14, CS15, CS16, CS17, CS18, CS19, CS2, CS20, CS21, CS22, CS23, CS24, CS25, CS26, CS27, CS28, CS29, CS3, CS30, CS31, CS32, CS33, CS34, CS35, CS36, CS37, CS38, CS39, CS4, CS40, CS41, CS42, CS43, CS44, CS45, CS46, CS47, CS48, CS49, CS5, CS50, CS51, CS52, CS53, CS54, CS55, CS56, CS57, CS58, CS59, CS6, CS60, CS61, CS62, CS63, CS64, CS65, CS66, CS67, CS68, CS69, CS7, CS70, CS71, CS72, CS73, CS74, CS75, CS76, CS77, CS78, CS79, CS8, CS80, CS81, CS82, CS83, CS84, CS85, CS86, CS87, CS9, CS? (x16): 0.1uF, Capacitor_SMD:C_0805_2012Metric_Pad1.15x1.40mm_HandSolder, symbol Device:C_Small
- added E? (x16): SK6812MINI-E, Components:SK6812B-SIDE, symbol Components:SK6812MINI-E
- D1, D10, D11, D12, D13, D14, D15, D16, D17, D18, D19, D2, D20, D21, D22, D23, D24, D25, D26, D27, D28, D29, D3, D30, D31, D32, D33, D34, D35, D36, D37, D38, D39, D4, D40, D41, D42, D43, D44, D45, D46, D47, D48, D49, D5, D50, D51, D52, D53, D54, D55, D56, D57, D58, D59, D6, D60, D61, D62, D63, D64, D65, D66, D67, D68, D69, D7, D70, D71, D72, D73, D74, D75, D76, D79, D8, D80, D81, D82, D83, D86, D9, D90, D91, D92, D93, D94, D95, D96: JLC (none) -> SOD-323F; LCSC (none) -> C2128
- D97: JLC (none) -> SOD-123; LCSC (none) -> C260260
- L3: JLC (none) -> SMD-2.4x2.4x1.1; LCSC (none) -> C89149
- Q1: JLC (none) -> SOT-23-3; LCSC (none) -> C150470
- Q2: value DM2305 -> DMG2305; JLC (none) -> SOT-23-3; LCSC (none) -> C150470
- Q3: JLC (none) -> SOT-23-3; LCSC (none) -> C8545
- U3, U4: JLC (none) -> TSSOP-16; LCSC (none) -> C5948
- U5: JLC (none) -> SOT-23-5; LCSC (none) -> C14879
- U6: JLC (none) -> SOT-23-5; LCSC (none) -> C201586
- gave numbers to parts that had none: 1
Connections:
- net GND: now also CS10.1, CS11.1, CS12.1, CS13.1, CS14.1, CS15.1, CS16.1, CS17.1, CS18.1, CS19.1, CS2.1, CS20.1, CS21.1, CS22.1, CS23.1, CS24.1, CS25.1, CS26.1, CS27.1, CS28.1, CS29.1, CS3.1, CS30.1, CS31.1, CS32.1, CS33.1, CS34.1, CS35.1, CS36.1, CS37.1, CS38.1, CS39.1, CS4.1, CS40.1, CS41.1, CS42.1, CS43.1, CS44.1, CS45.1, CS46.1, CS47.1, CS48.1, CS49.1, CS5.1, CS50.1, CS51.1, CS52.1, CS53.1, CS54.1, CS55.1, CS56.1, CS57.1, CS58.1, CS59.1, CS6.1, CS60.1, CS61.1, CS62.1, CS63.1, CS64.1, CS65.1, CS66.1, CS67.1, CS68.1, CS69.1, CS7.1, CS70.1, CS71.1, CS72.1, CS73.1, CS74.1, CS75.1, CS76.1, CS77.1, CS78.1, CS79.1, CS8.1, CS80.1, CS81.1, CS82.1, CS83.1, CS84.1, CS85.1, CS86.1, CS87.1, CS9.1, CS?.1, CS?.1, CS?.1, CS?.1, CS?.1, CS?.1, CS?.1, CS?.1, CS?.1, CS?.1, CS?.1, CS?.1, CS?.1, CS?.1, CS?.1, CS?.1, E?.3 (GND), E?.3 (GND), E?.3 (GND), E?.3 (GND), E?.3 (GND), E?.3 (GND), E?.3 (GND), E?.3 (GND), E?.3 (GND), E?.3 (GND), E?.3 (GND), E?.3 (GND), E?.3 (GND), E?.3 (GND), E?.3 (GND), E?.3 (GND)
- net LED_VDD: now also CS10.2, CS11.2, CS12.2, CS13.2, CS14.2, CS15.2, CS16.2, CS17.2, CS18.2, CS19.2, CS2.2, CS20.2, CS21.2, CS22.2, CS23.2, CS24.2, CS25.2, CS26.2, CS27.2, CS28.2, CS29.2, CS3.2, CS30.2, CS31.2, CS32.2, CS33.2, CS34.2, CS35.2, CS36.2, CS37.2, CS38.2, CS39.2, CS4.2, CS40.2, CS41.2, CS42.2, CS43.2, CS44.2, CS45.2, CS46.2, CS47.2, CS48.2, CS49.2, CS5.2, CS50.2, CS51.2, CS52.2, CS53.2, CS54.2, CS55.2, CS56.2, CS57.2, CS58.2, CS59.2, CS6.2, CS60.2, CS61.2, CS62.2, CS63.2, CS64.2, CS65.2, CS66.2, CS67.2, CS68.2, CS69.2, CS7.2, CS70.2, CS71.2, CS72.2, CS73.2, CS74.2, CS75.2, CS76.2, CS77.2, CS78.2, CS79.2, CS8.2, CS80.2, CS81.2, CS82.2, CS83.2, CS84.2, CS85.2, CS86.2, CS87.2, CS9.2, CS?.2, CS?.2, CS?.2, CS?.2, CS?.2, CS?.2, CS?.2, CS?.2, CS?.2, CS?.2, CS?.2, CS?.2, CS?.2, CS?.2, CS?.2, CS?.2, E?.1 (VDD), E?.1 (VDD), E?.1 (VDD), E?.1 (VDD), E?.1 (VDD), E?.1 (VDD), E?.1 (VDD), E?.1 (VDD), E?.1 (VDD), E?.1 (VDD), E?.1 (VDD), E?.1 (VDD), E?.1 (VDD), E?.1 (VDD), E?.1 (VDD), E?.1 (VDD)
- net LED_SERIAL_8: now reaches E87.2 (DOUT)
- net LED_SERIAL_8: now also E?.4 (DIN)
- new net: E?.2 (DOUT), E?.4 (DIN) (x15)
Other:
- moved on the sheet: CS1, Q2, Q3, R10, R2, R3

Commit message: More keyboard documentation and polishing.
Parts:
- added FID1, FID2, FID3, FID4, FID5, FID6, FID7, FID8: Fiducial, Fiducial:Fiducial_1mm_Mask2mm, symbol Mechanical:Fiducial
- added J5: Conn_01x02, Connector_PinHeader_2.54mm:PinHeader_1x02_P2.54mm_Vertical, symbol Connector_Generic:Conn_01x02
- CS100, CS101, CS102, CS103, CS88, CS89, CS90, CS91, CS92, CS93, CS94, CS95, CS96, CS97, CS98, CS99: renamed from CS?; footprint Capacitor_SMD:C_0805_2012Metric_Pad1.15x1.40mm_HandSolder -> Capacitor_SMD:C_0603_1608Metric_Pad1.05x0.95mm_HandSolder
- gave numbers to parts that had none: 16
Connections:
- net KEY_X15: now also SW63.1; no longer SW63.2
- net KEY_X_REGISTER_CLK: now also J5.1 (Pin_1)
- net KEY_X_SERIAL_CLK: now also J5.2 (Pin_2)
- net at D63.2 (A): now also SW63.2; no longer SW63.1
Other:
- note added: "Charge Current Resistor\n10K = 100mA\n5K = 200mA\n2K = 500mA\n1K = 1000mA"
- moved on the sheet: SW63
