File: pkg/things/fan_controller/boards/board-hl15-latest/board-hl15-latest.kicad_sch (KiCad schematic)
At the start: 14 parts, among them J1 FAN1, J2 FAN2, J3 FAN3, J4 FAN4, J5 FAN5, J6 FAN6, J7 FAN7, J8 FAN8, J9 POWER, Q1 2N7002, Q2 2N7002, Q3 2N7002, Q4 2N7002, U1 NRF52840_ITSY_BITSY

Commit message: Some cleanup of local changes.
Other:
- note added: "TODO: D7 is P1.08"
- note added: "TODO: Filter cap on the tachometer."
- note added: "TODO: Pull down all PWMs with 10K resistors. (this way we don't need the microcontroller to init to ensure we are running at 100%)."
Changed lines of the file:
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@@
     (stroke (width 0) (type default))
+  )
+  (text "TODO: Filter cap on the tachometer." (at 68.58 77.47 0)
+    (effects (font (size 1.27 1.27)) (justify left bottom))
+  )
+  (text "TODO: D7 is P1.08" (at 104.14 90.17 0)
+    (effects (font (size 1.27 1.27)) (justify left bottom))
+  )
+  (text "TODO: Pull down all PWMs with 10K resistors.\n(this way we don't need the microcontroller to init to ensure we are running at 100%)."
+    (at 60.96 71.12 0)
+    (effects (font (size 1.27 1.27)) (justify left bottom))
   )
   (global_label "FAN_C_PWM" (shape input) (at 124.46 124.46 0) (fields_autoplaced)
@@
       (effects (font (size 1.27 1.27)) (justify left) hide)
     )
+  )
+  (global_label "TODO: Need a CMOS-inverter type circuit to drive the PWM both high and low." (shape input)
+    (at 55.88 82.55 0) (fields_autoplaced)
+    (effects (font (size 1.27 1.27)) (justify left))
+    (property "Intersheetrefs" "${INTERSHEET_REFS}" (at 135.7902 82.55 0)
+      (effects (font (size 1.27 1.27)) (justify left) hide)
+    )
