File: pkg/cnc/boards/voron_v0_bed/board-latest/board-latest.kicad_pcb (KiCad board)
At the start: 2 copper layers, 38.4 x 34.1 mm, 11 parts, among them J1 BED_TEMP, J2 FAN1, J3 LED, J4 INPUT, J5 FAN2, Q1 AO3400A, Q2 AO3400A, U1 ATtiny412-SS

Commit message: Lot's of kicad and cluster improvements.
Parts:
- removed J5: FAN2, Connector_JST:JST_SH_BM03B-SRSS-TB_1x03-1MP_P1.00mm_Vertical
- removed Q2: AO3400A, Package_TO_SOT_SMD:SOT-23
- added J6: AUX_TEMP, Connector_JST:JST_SH_SM02B-SRSS-TB_1x02-1MP_P1.00mm_Horizontal, F.Cu at (124.4, 121.6)
- added R1: 4.7K, Resistor_SMD:R_0603_1608Metric_Pad0.98x0.95mm_HandSolder, F.Cu at (124.0, 114.8)
- added R2: 10K, Resistor_SMD:R_0603_1608Metric_Pad0.98x0.95mm_HandSolder, F.Cu at (124.0, 116.6)
Connections:
- net FAN2_PWM renamed LED_SERIAL
- U1 pad 5: FAN2_TACH -> AUX_TEMP_SENSE
Routing:
- net FAN2_TACH: track 15.9 -> 0.00 mm
- net LED_SERIAL: track 14.1 -> 7.37 mm
- net Net-(J6-Pin_2): track 0.00 -> 4.79 mm
- net AUX_TEMP_SENSE: track 0.00 -> 3.96 mm
- net FAN2_LOW: track 3.73 -> 0.00 mm
- net +5V: track 53.8 -> 50.6 mm
Other:
- board size 38.4 x 34.1 mm -> 38.3 x 34.1 mm

Commit message: Lot's of changes.
Parts:
- added C1: 4.7nF 10V, Capacitor_SMD:C_0603_1608Metric_Pad1.08x0.95mm_HandSolder, F.Cu at (115.0, 106.9)
- added J5: SHEET_TEMP, Connector_JST:JST_SH_SM02B-SRSS-TB_1x02-1MP_P1.00mm_Horizontal, F.Cu at (112.8, 121.4)
- added R3: 4.7K, Resistor_SMD:R_0603_1608Metric_Pad0.98x0.95mm_HandSolder, F.Cu at (112.0, 116.8)
- added R6: 10K, Resistor_SMD:R_0603_1608Metric_Pad0.98x0.95mm_HandSolder, F.Cu at (111.9, 115.1)
- added TP1: TestPoint, TestPoint:TestPoint_Pad_D1.0mm, F.Cu at (122.3, 116.6)
- J4: footprint Connector_JST:JST_SH_BM03B-SRSS-TB_1x03-1MP_P1.00mm_Vertical -> Connector_JST:JST_PH_B3B-PH-SM4-TB_1x03-1MP_P2.00mm_Vertical
- moved J1 2.57 mm to (124.4, 99.6)
- moved Q1 2.13 mm to (118.4, 106.7)
- moved J3 1.89 mm to (119.4, 121.4)
- moved C5 1.80 mm to (109.8, 106.6)
- moved J2 1.69 mm to (118.0, 100.5), turned to 180 degrees
- moved J6 1.57 mm to (126.0, 121.4)
- moved R1 1.40 mm to (125.3, 114.7)
- moved R2 1.40 mm to (125.3, 116.6)
- moved J4 1.17 mm to (108.8, 101.9)
Connections:
- Q1 pad 1: FAN1_PWM -> LED_SERIAL
- U1 pad 2: FAN_PWM -> HOST_SERIAL
- U1 pad 4: HOST_SERIAL -> SHEET_TEMP_SENSE
- U1 pad 5: AUX_TEMP_SENSE -> LED_SERIAL
- U1 pad 6: LED_SERIAL -> AUX_TEMP_SENSE
Routing:
- net +5V: track 50.6 -> 65.6 mm, vias 4 -> 3
- net GND: track 20.2 -> 34.1 mm, vias 5 -> 4
- net FAN_PWM: track 6.46 -> 0.00 mm
- net LED_SERIAL: track 7.37 -> 13.7 mm
- net Net-(J5-Pin_2): track 0.00 -> 5.52 mm
- net FAN1_LOW: track 2.36 -> 6.03 mm
- net FAN1_TACH: track 12.3 -> 16.0 mm
- net Net-(J1-Pin_2): track 4.74 -> 7.60 mm
- net AUX_TEMP_SENSE: track 3.96 -> 6.56 mm
- net SHEET_TEMP_SENSE: track 0.00 -> 2.14 mm
- net HOST_SERIAL: track 15.0 -> 15.5 mm

Commit message: Flush some changes
Parts:
- added C2: 0.1uF 10V, Capacitor_SMD:C_0603_1608Metric_Pad1.08x0.95mm_HandSolder, F.Cu at (114.1, 109.0)
- R1, R3, R4: value 4.7K -> 1K (0.1%)
Routing:
- net +5V: track 65.6 -> 68.2 mm
- net GND: track 34.1 -> 36.6 mm
- net HOST_SERIAL: track 15.5 -> 16.1 mm
Changed lines of the file:
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@@
         (effects (font (size 1 1) (thickness 0.15)))
     )
-    (fp_text value "4.7K" (at 0 1.43) (layer "F.Fab") hide
+    (fp_text value "1K (0.1%)" (at 0 1.43) (layer "F.Fab") hide
         (effects (font (size 1 1) (thickness 0.15)))
     )
@@
         (effects (font (size 1 1) (thickness 0.15)))
     )
-    (fp_text value "4.7K" (at 0 1.43) (layer "F.Fab") hide
+    (fp_text value "1K (0.1%)" (at 0 1.43) (layer "F.Fab") hide
         (effects (font (size 1 1) (thickness 0.15)))
     )
@@
         (effects (font (size 1 1) (thickness 0.15)))
     )
-    (fp_text value "4.7K" (at 0 1.43) (layer "F.Fab") hide
+    (fp_text value "1K (0.1%)" (at 0 1.43) (layer "F.Fab") hide
         (effects (font (size 1 1) (thickness 0.15)))
     )
@@
     (pad "MP" smd roundrect (at 1.8 1.875) (size 1.2 1.8) (layers "F.Cu" "F.Paste" "F.Mask") (roundrect_rratio 0.208333))
     (model "${KICAD7_3DMODEL_DIR}/Connector_JST.3dshapes/JST_SH_SM02B-SRSS-TB_1x02-1MP_P1.00mm_Horizontal.wrl"
+      (offset (xyz 0 0 0))
+      (scale (xyz 1 1 1))
+      (rotate (xyz 0 0 0))
+    )
+  )
+  (footprint "Capacitor_SMD:C_0603_1608Metric_Pad1.08x0.95mm_HandSolder" (layer "F.Cu")
+    (at 114.1 108.99 180)
+    (descr "Capacitor SMD 0603 (1608 Metric), square (rectangular) end terminal, IPC_7351 nominal with elongated pad for handsoldering. (Body size source: IPC-SM-782 page 76, https://www.pcb-3d.com/wordpress/wp-content/uploads/ipc-sm-782a_amendment_1_and_2.pdf), generated with kicad-footprint-generator")
+    (tags "capacitor handsolder")
+    (property "Sheetfile" "board-latest.kicad_sch")
+    (property "Sheetname" "")
+    (property "ki_description" "Unpolarized capacitor, small symbol")
+    (property "ki_keywords" "capacitor cap")
+    (attr smd)
+    (fp_text reference "C2" (at 0 -1.43) (layer "F.SilkS") hide
+        (effects (font (size 1 1) (thickness 0.15)))
+    )
+    (fp_text value "0.1uF 10V" (at 0 1.43) (layer "F.Fab") hide
+        (effects (font (size 1 1) (thickness 0.15)))
+    )
+    (fp_text user "${REFERENCE}" (at 0 0) (layer "F.Fab") hide
+        (effects (font (size 0.4 0.4) (thickness 0.06)))
+    )
+    (fp_line (start -0.146267 -0.51) (end 0.146267 -0.51)
+      (stroke (width 0.12) (type solid)) (layer "F.SilkS"))
+    (fp_line (start -0.146267 0.51) (end 0.146267 0.51)
+      (stroke (width 0.12) (type solid)) (layer "F.SilkS"))
+    (fp_line (start -1.65 -0.73) (end 1.65 -0.73)
+      (stroke (width 0.05) (type solid)) (layer "F.CrtYd"))
+    (fp_line (start -1.65 0.73) (end -1.65 -0.73)
+      (stroke (width 0.05) (type solid)) (layer "F.CrtYd"))
+    (fp_line (start 1.65 -0.73) (end 1.65 0.73)
+      (stroke (width 0.05) (type solid)) (layer "F.CrtYd"))
+    (fp_line (start 1.65 0.73) (end -1.65 0.73)
+      (stroke (width 0.05) (type solid)) (layer "F.CrtYd"))
+    (fp_line (start -0.8 -0.4) (end 0.8 -0.4)
+      (stroke (width 0.1) (type solid)) (layer "F.Fab"))
+    (fp_line (start -0.8 0.4) (end -0.8 -0.4)
+      (stroke (width 0.1) (type solid)) (layer "F.Fab"))
+    (fp_line (start 0.8 -0.4) (end 0.8 0.4)
+      (stroke (width 0.1) (type solid)) (layer "F.Fab"))
+    (fp_line (start 0.8 0.4) (end -0.8 0.4)
+      (stroke (width 0.1) (type solid)) (layer "F.Fab"))
+    (pad "1" smd roundrect (at -0.8625 0 180) (size 1.075 0.95) (layers "F.Cu" "F.Paste" "F.Mask") (roundrect_rratio 0.25)
+      (net 2 "+5V") (pintype "passive"))
+    (pad "2" smd roundrect (at 0.8625 0 180) (size 1.075 0.95) (layers "F.Cu" "F.Paste" "F.Mask") (roundrect_rratio 0.25)
+      (net 7 "GND") (pintype "passive"))
+    (model "${KICAD6_3DMODEL_DIR}/Capacitor_SMD.3dshapes/C_0603_1608Metric.wrl"
       (offset (xyz 0 0 0))
       (scale (xyz 1 1 1))
@@
   (segment (start 124.35 106.1975) (end 124.5625 106.41) (width 0.4) (layer "F.Cu") (net 1))
   (segment (start 117.424238 97.663) (end 117.97 98.208762) (width 0.8) (layer "F.Cu") (net 2))
-  (segment (start 114.92 110.1) (end 114.92 111.2) (width 0.4) (layer "F.Cu") (net 2))
-  (segment (start 108.9475 107.1695) (end 108.9475 106.58) (width 0.8) (layer "F.Cu") (net 2))
+  (segment (start 108.9475 107.7775) (end 108.9475 106.58) (width 0.8) (layer "F.Cu") (net 2))
   (segment (start 118.470001 97.915) (end 117.97 98.415001) (width 0.4) (layer "F.Cu") (net 2))
   (segment (start 108.77 99.89) (end 108.77 102.38) (width 0.4) (layer "F.Cu") (net 2))
@@
   (segment (start 119.393394 97.915) (end 118.470001 97.915) (width 0.4) (layer "F.Cu") (net 2))
   (segment (start 117.51 117.59) (end 117.268 117.348) (width 0.4) (layer "F.Cu") (net 2))
+  (segment (start 114.9625 108.99) (end 114.9625 111.1575) (width 0.4) (layer "F.Cu") (net 2))
   (segment (start 118.618 117.348) (end 119.396 118.126) (width 0.8) (layer "F.Cu") (net 2))
   (segment (start 117.094 117.348) (end 116.586 116.84) (width 0.4) (layer "F.Cu") (net 2))
@@
   (segment (start 108.9475 106.58) (end 108.9475 102.5575) (width 0.8) (layer "F.Cu") (net 2))
   (segment (start 116.586 116.84) (end 112.9265 116.84) (width 0.4) (layer "F.Cu") (net 2))
-  (segment (start 110.236 108.458) (end 108.9475 107.1695) (width 0.8) (layer "F.Cu") (net 2))
   (segment (start 110.997 97.663) (end 117.424238 97.663) (width 0.8) (layer "F.Cu") (net 2))
   (segment (start 117.268 117.348) (end 117.094 117.348) (width 0.4) (layer "F.Cu") (net 2))
@@
   (segment (start 117.094 117.348) (end 118.618 117.348) (width 0.8) (layer "F.Cu") (net 2))
   (segment (start 122.7375 106.41) (end 121.37 105.0425) (width 0.4) (layer "F.Cu") (net 2))
-  (segment (start 113.57 108.75) (end 114.92 110.1) (width 0.4) (layer "F.Cu") (net 2))
-  (segment (start 113.278 108.458) (end 110.236 108.458) (width 0.8) (layer "F.Cu") (net 2))
-  (segment (start 113.57 108.75) (end 113.278 108.458) (width 0.4) (layer "F.Cu") (net 2))
+  (segment (start 114.9625 111.1575) (end 114.92 111.2) (width 0.4) (layer "F.Cu") (net 2))
+  (segment (start 112.04 110.87) (end 108.9475 107.7775) (width 0.8) (layer "F.Cu") (net 2))
   (segment (start 108.9475 102.5575) (end 108.77 102.38) (width 0.4) (layer "F.Cu") (net 2))
+  (segment (start 112.04 110.87) (end 114.59 110.87) (width 0.4) (layer "F.Cu") (net 2))
+  (segment (start 114.59 110.87) (end 114.92 111.2) (width 0.4) (layer "F.Cu") (net 2))
   (via (at 122.682 113.03) (size 2) (drill 0.9) (layers "F.Cu" "B.Cu") (net 2))
-  (via (at 113.57 108.75) (size 2) (drill 0.9) (layers "F.Cu" "B.Cu") (net 2))
+  (via (at 112.04 110.87) (size 2) (drill 0.9) (layers "F.Cu" "B.Cu") (net 2))
   (via (at 117.094 117.348) (size 2) (drill 0.9) (layers "F.Cu" "B.Cu") (net 2))
-  (segment (start 113.57 108.75) (end 114.06 108.75) (width 0.4) (layer "B.Cu") (net 2))
   (segment (start 118.34 113.03) (end 117.52 112.21) (width 1.2) (layer "B.Cu") (net 2))
+  (segment (start 112.14 110.97) (end 116.28 110.97) (width 1.2) (layer "B.Cu") (net 2))
+  (segment (start 116.28 110.97) (end 117.52 112.21) (width 1.2) (layer "B.Cu") (net 2))
+  (segment (start 112.04 110.87) (end 112.14 110.97) (width 1.2) (layer "B.Cu") (net 2))
   (segment (start 117.094 117.348) (end 117.52 116.922) (width 0.8) (layer "B.Cu") (net 2))
   (segment (start 117.52 116.922) (end 117.52 112.21) (width 1.2) (layer "B.Cu") (net 2))
   (segment (start 122.682 113.03) (end 118.34 113.03) (width 1.2) (layer "B.Cu") (net 2))
-  (segment (start 114.06 108.75) (end 117.52 112.21) (width 1.2) (layer "B.Cu") (net 2))
   (segment (start 116.97 105.407) (end 116.395 105.982) (width 0.4) (layer "F.Cu") (net 3))
   (segment (start 116.97 99.19) (end 116.97 105.407) (width 0.4) (layer "F.Cu") (net 3))
@@
   (segment (start 117.48 113.594999) (end 118.895001 115.01) (width 0.4) (layer "F.Cu") (net 5))
   (segment (start 120.396 119.38) (end 120.396 115.536) (width 0.4) (layer "F.Cu") (net 5))
-  (segment (start 106.77 107.834999) (end 106.77 102.38) (width 0.4) (layer "F.Cu") (net 6))
-  (segment (start 111.405001 112.47) (end 106.77 107.834999) (width 0.4) (layer "F.Cu") (net 6))
-  (segment (start 114.92 112.47) (end 111.405001 112.47) (width 0.4) (layer "F.Cu") (net 6))
+  (segment (start 114.92 112.47) (end 110.38 112.47) (width 0.4) (layer "F.Cu") (net 6))
+  (segment (start 110.38 112.47) (end 106.77 108.86) (width 0.4) (layer "F.Cu") (net 6))
+  (segment (start 106.77 108.86) (end 106.77 102.38) (width 0.4) (layer "F.Cu") (net 6))
   (segment (start 114.1741 106.8832) (end 113.6142 106.8832) (width 0.4) (layer "F.Cu") (net 7))
   (segment (start 110.77 102.38) (end 110.77 106.4825) (width 0.8) (layer "F.Cu") (net 7))
@@
   (segment (start 124.336 120.904) (end 125.4 119.84) (width 0.8) (layer "F.Cu") (net 7))
   (segment (start 119.87 111.08) (end 119.88 111.09) (width 0.8) (layer "F.Cu") (net 7))
+  (segment (start 113.2375 107.8198) (end 114.1741 106.8832) (width 0.4) (layer "F.Cu") (net 7))
   (segment (start 123.91 100.95) (end 123.91 102.83) (width 0.4) (layer "F.Cu") (net 7))
   (segment (start 123.19 118.618) (end 124.73 118.618) (width 0.8) (layer "F.Cu") (net 7))
@@
   (segment (start 120.904 109.22) (end 119.38 107.696) (width 0.8) (layer "F.Cu") (net 7))
   (segment (start 119.38 107.696) (end 119.38 107.6275) (width 0.4) (layer "F.Cu") (net 7))
+  (segment (start 113.2375 108.99) (end 113.2375 107.8198) (width 0.4) (layer "F.Cu") (net 7))
   (segment (start 123.91 102.83) (end 123.11 103.63) (width 0.4) (layer "F.Cu") (net 7))
   (segment (start 118.396 120.655) (end 118.396 119.874) (width 0.8) (layer "F.Cu") (net 7))
