File: pkg/cnc/boards/voron_v0_bed/board-latest/board-latest.kicad_sch (KiCad schematic)
At the start: 11 parts, among them J1 BED_TEMP, J2 FAN1, J3 LED, J4 INPUT, J5 FAN2, Q1 AO3400A, Q2 AO3400A, U1 ATtiny412-SS

Commit message: Lot's of kicad and cluster improvements.
Parts:
- removed J5: FAN2, Connector_JST:JST_SH_BM03B-SRSS-TB_1x03-1MP_P1.00mm_Vertical, symbol Connector_Generic:Conn_01x03
- removed Q2: AO3400A, Package_TO_SOT_SMD:SOT-23, symbol Transistor_FET:AO3400A
- added J6: AUX_TEMP, Connector_JST:JST_SH_SM02B-SRSS-TB_1x02-1MP_P1.00mm_Horizontal, symbol Connector_Generic:Conn_01x02
- added R1: 4.7K, Resistor_SMD:R_0603_1608Metric_Pad0.98x0.95mm_HandSolder, symbol Device:R_Small
- added R2: 10K, Resistor_SMD:R_0603_1608Metric_Pad0.98x0.95mm_HandSolder, symbol Device:R_Small
Connections:
- net +5V: now also R1.2
- net GND: now also J6.1 (Pin_1)
- net FAN2_PWM renamed LED_SERIAL
- net FAN2_TACH renamed AUX_TEMP_SENSE
- net AUX_TEMP_SENSE: now also R2.1
- new net: J6.2 (Pin_2), R1.1, R2.2
Other:
- moved on the sheet: J1, J3, R4, R5

Commit message: Lot's of changes.
Parts:
- added C1: 4.7nF 10V, Capacitor_SMD:C_0603_1608Metric_Pad1.08x0.95mm_HandSolder, symbol Device:C_Small
- added J5: SHEET_TEMP, Connector_JST:JST_SH_SM02B-SRSS-TB_1x02-1MP_P1.00mm_Horizontal, symbol Connector_Generic:Conn_01x02
- added R3: 4.7K, Resistor_SMD:R_0603_1608Metric_Pad0.98x0.95mm_HandSolder, symbol Device:R_Small
- added R6: 10K, Resistor_SMD:R_0603_1608Metric_Pad0.98x0.95mm_HandSolder, symbol Device:R_Small
- added TP1: TestPoint, TestPoint:TestPoint_Pad_D1.0mm, symbol Connector:TestPoint
- J4: footprint Connector_JST:JST_SH_BM03B-SRSS-TB_1x03-1MP_P1.00mm_Vertical -> Connector_JST:JST_PH_B3B-PH-SM4-TB_1x03-1MP_P2.00mm_Vertical
Connections:
- net FAN1_PWM is gone; now on net LED_SERIAL: Q1.1 (G)
- net FAN_PWM is gone; now on net HOST_SERIAL: U1.2 (PA6)
- net +5V: now also R3.2
- net AUX_TEMP_SENSE: now also U1.6 (~{RESET}/PA0), TP1.1; no longer U1.5 (PA2)
- net FAN1_TACH: now also C1.1
- net GND: now also C1.2, J5.1 (Pin_1)
- net HOST_SERIAL: no longer U1.4 (PA1)
- net LED_SERIAL: now also U1.5 (PA2); no longer U1.6 (~{RESET}/PA0)
- new net: J5.2 (Pin_2), R3.1, R6.2
- new net SHEET_TEMP_SENSE: R6.1, U1.4 (PA1)
Other:
- note added: "Analog input (_SENSE) signals can be on any pin."
- note added: "HOST_SERIAL must be connected to a TXD pin for one-wire serial. (PA1 or PA6)"

Commit message: Flush some changes
Parts:
- added C2: 0.1uF 10V, Capacitor_SMD:C_0603_1608Metric_Pad1.08x0.95mm_HandSolder, symbol Device:C_Small
- R1, R3, R4: value 4.7K -> 1K (0.1%)
Connections:
- net +5V: now also C2.1
- net GND: now also C2.2
Changed lines of the file:
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@@
+    (stroke (width 0) (type default))
+  )
+  (wire (pts (xy 53.34 52.07) (xy 53.34 54.61))
     (stroke (width 0) (type default))
   )
@@
   )
   (wire (pts (xy 34.29 59.69) (xy 34.29 62.23))
+    (stroke (width 0) (type default))
+  )
+  (wire (pts (xy 53.34 59.69) (xy 53.34 62.23))
     (stroke (width 0) (type default))
   )
@@
       (effects (font (size 1.27 1.27)) (justify right))
     )
-    (property "Value" "4.7K" (at 140.081 90.932 0)
+    (property "Value" "1K (0.1%)" (at 147.32 88.9 0)
       (effects (font (size 1.27 1.27)) (justify right))
     )
@@
       (effects (font (size 1.27 1.27)) (justify right))
     )
-    (property "Value" "4.7K" (at 133.731 137.922 0)
+    (property "Value" "1K (0.1%)" (at 140.97 135.89 0)
       (effects (font (size 1.27 1.27)) (justify right))
     )
@@
       (effects (font (size 1.27 1.27)) (justify right))
     )
-    (property "Value" "4.7K" (at 128.651 168.402 0)
+    (property "Value" "1K (0.1%)" (at 135.89 166.37 0)
       (effects (font (size 1.27 1.27)) (justify right))
     )
@@
         )
       )
+    )
+  )
+  (symbol (lib_id "power:+5V") (at 53.34 52.07 0) (unit 1)
+    (in_bom yes) (on_board yes) (dnp no) (fields_autoplaced)
+    (property "Reference" "#PWR018" (at 53.34 55.88 0)
+      (effects (font (size 1.27 1.27)) hide)
+    )
+    (property "Value" "+5V" (at 53.34 46.99 0)
+      (effects (font (size 1.27 1.27)))
+    )
+    (property "Footprint" "" (at 53.34 52.07 0)
+      (effects (font (size 1.27 1.27)) hide)
+    )
+    (property "Datasheet" "" (at 53.34 52.07 0)
+      (effects (font (size 1.27 1.27)) hide)
+    )
+    (pin "1")
+    (instances
+      (project "board-latest"
+        (path "/1b0ea594-0486-47a9-a46b-c33a533a619b"
+          (reference "#PWR018") (unit 1)
+        )
+      )
+    )
+  )
+  (symbol (lib_id "Device:C_Small") (at 53.34 57.15 0) (unit 1)
+    (in_bom yes) (on_board yes) (dnp no)
+    (property "Reference" "C2" (at 48.26 55.88 0)
+      (effects (font (size 1.27 1.27)) (justify left))
+    )
+    (property "Value" "0.1uF 10V" (at 40.64 58.42 0)
+      (effects (font (size 1.27 1.27)) (justify left))
+    )
+    (property "Footprint" "Capacitor_SMD:C_0603_1608Metric_Pad1.08x0.95mm_HandSolder" (at 53.34 57.15 0)
+      (effects (font (size 1.27 1.27)) hide)
+    )
+    (property "Datasheet" "~" (at 53.34 57.15 0)
+      (effects (font (size 1.27 1.27)) hide)
+    )
+    (pin "1")
+    (pin "2")
+    (instances
+      (project "board-latest"
+        (path "/1b0ea594-0486-47a9-a46b-c33a533a619b"
+          (reference "C2") (unit 1)
+        )
+      )
+    )
+  )
+  (symbol (lib_id "power:GND") (at 53.34 62.23 0) (unit 1)
+    (in_bom yes) (on_board yes) (dnp no)
+    (property "Reference" "#PWR019" (at 53.34 68.58 0)
+      (effects (font (size 1.27 1.27)) hide)
+    )
+    (property "Value" "GND" (at 53.467 66.6242 0)
+      (effects (font (size 1.27 1.27)))
+    )
+    (property "Footprint" "" (at 53.34 62.23 0)
+      (effects (font (size 1.27 1.27)) hide)
+    )
+    (property "Datasheet" "" (at 53.34 62.23 0)
+      (effects (font (size 1.27 1.27)) hide)
+    )
+    (pin "1")
+    (instances
+      (project "board-latest"
+        (path "/1b0ea594-0486-47a9-a46b-c33a533a619b"
+          (reference "#PWR019") (unit 1)
+        )
+      )
