File: pkg/cnc/boards/voron_v0_toolhead/board-latest/board-latest.kicad_pcb (KiCad board)
At the start: 4 copper layers, 52.5 x 46.5 mm, 77 parts, among them J1 Conn_02x03_Odd_Even, J10 FAN, J11 LED, J12 LED, J13 Conn_01x01, J2 UMB, J3 TEMP, J4 PROBE, J5 HEAT, J6 FIL, J7 STEP, J8 FAN, J9 FAN, Q1 BSS138, Q2 AON7524, Q4 AO3400A, Q5 AO3400A, Q6 AO3400A, SW2 USR, U1 AP2112K-3.3, U2 MA732, U3 AP63205WU, U5 BMD-380-A-R, U6 LIS2DH, U7 SK6812MINI-E, U8 TMC2209-LA

Commit message: Flush some changes
Other:
- board text added: "TODO: Smaller fill clearance / reduce 24V -> TMC resistance"
- board text added: "V0 Tool R?"
- board text removed: "V0 Tool R1"
Changed lines of the file:
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@@
   (gr_rect (start 104.92 120.55167) (end 113.22 126.85167)
     (stroke (width 0.2) (type default)) (fill none) (layer "User.1"))
-  (gr_rect (start 104.92 131.57467) (end 138.92 126.85167)
+  (gr_rect (start 104.92 126.85167) (end 138.92 131.57467)
     (stroke (width 0.2) (type default)) (fill none) (layer "User.1"))
   (gr_rect (start 95.67 96.25) (end 148.17 103.75)
@@
   (gr_line (start 144.42 120.55167) (end 144.42 125)
     (stroke (width 0.15) (type default)) (layer "User.1"))
-  (gr_text "V0 Tool R1" (at 142.575 109.85 -90) (layer "F.SilkS")
+  (gr_text "V0 Tool R?" (at 142.575 109.85 270) (layer "F.SilkS")
     (effects (font (size 1 1) (thickness 0.15)) (justify left bottom))
   )
+  (gr_text "TODO: Smaller fill clearance / reduce 24V -> TMC resistance" (at 116.459 79.375) (layer "F.Fab")
+    (effects (font (size 1 1) (thickness 0.15)) (justify left bottom))
+  )
