File: pkg/cnc/boards/voron_v0_toolhead/board-latest/motor.kicad_sch (KiCad schematic)
At the start: 16 parts, among them J13 Conn_01x01, J7 STEP, U2 MA732, U8 TMC2209-LA

Commit message: Flush some changes
Other:
- note added: "TODO: Remove solder mask for heatsink."
Changed lines of the file:
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@@
+    (effects (font (size 1.27 1.27)) (justify left bottom))
+  )
+  (text "TODO: Remove solder mask for heatsink." (at 44.45 69.85 0)
     (effects (font (size 1.27 1.27)) (justify left bottom))
   )
