File: pkg/cnc/boards/voron_v0_toolhead/board-latest/board-latest.kicad_sch (KiCad schematic)
At the start: 11 parts, among them J1 Conn_02x03_Odd_Even, J2 UMB, J6 FIL, U5 BMD-380-A-R

Commit message: Flush some changes
Parts:
- R3, R4: value 22 -> 27
Other:
- note added: "NOTE: The nRF52 REG0 can only do up to 25mA (5mA if radio is transmitting) So we don't use the REG0. Instead we directly feed 3.3V from an external LDO. Feeding both VCC/VCCH disables REG0. NOTE: 'Standard drive / low frequency' suggestions on pins are only relevant to radio performance."
- note added: "TODO: Switch everything to non-hand solder packages."
- note removed: "NOTE: The nRF52 REG0 can only do up to 25mA (5mA if radio is transmitting) So we don't use the REG0. Instead we directly feed 3.3V from an external LDO. NOTE: 'Standard drive / low frequency' suggestions on pins are only relevant to radio performance."
- note removed: "TODO: Figure out the factory REG0/1 settings for this."
Changed lines of the file:
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@@
+    (effects (font (size 1.27 1.27)) (justify left bottom))
+  )
+  (text "TODO: Switch everything to non-hand solder packages."
+    (at 120.65 26.67 0)
     (effects (font (size 1.27 1.27)) (justify left bottom))
   )
@@
     (effects (font (size 1.27 1.27)) (justify left bottom))
   )
-  (text "TODO: Figure out the factory REG0/1 settings for this."
-    (at 129.54 30.48 0)
-    (effects (font (size 1.27 1.27)) (justify left bottom))
-  )
   (text "NOTE: Should high drive all MOSFET PWM pins." (at 91.44 66.04 0)
     (effects (font (size 1.27 1.27)) (justify left bottom))
   )
-  (text "NOTE: The nRF52 REG0 can only do up to 25mA\n(5mA if radio is transmitting)\n\nSo we don't use the REG0. Instead we directly feed 3.3V\nfrom an external LDO.\n\nNOTE: 'Standard drive / low frequency' suggestions on pins are\nonly relevant to radio performance."
+  (text "NOTE: The nRF52 REG0 can only do up to 25mA\n(5mA if radio is transmitting)\n\nSo we don't use the REG0. Instead we directly feed 3.3V\nfrom an external LDO. Feeding both VCC/VCCH disables REG0.\n\nNOTE: 'Standard drive / low frequency' suggestions on pins are\nonly relevant to radio performance."
     (at 128.27 57.15 0)
     (effects (font (size 1.27 1.27)) (justify left bottom))
@@
       (effects (font (size 1.27 1.27)))
     )
-    (property "Value" "22" (at 38.227 41.402 90)
+    (property "Value" "27" (at 38.227 41.402 90)
       (effects (font (size 1.27 1.27)))
     )
@@
       (effects (font (size 1.27 1.27)))
     )
-    (property "Value" "22" (at 38.354 49.149 90)
-      (effects (font (size 1.27 1.27)))
-    )
+    (property "Value" "27" (at 38.354 49.149 90)
+      (effects (font (size 1.27 1.27)))
+    )

Commit message: Software improvements for the toolhead.
Other:
- note added: "TODO: Don't use P0.00/P0.01 since they are XTAL pins."
Changed lines of the file:
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@@
+    (effects (font (size 1.27 1.27)) (justify left bottom))
+  )
+  (text "TODO: Don't use P0.00/P0.01 since they are XTAL pins."
+    (at 69.85 95.25 0)
     (effects (font (size 1.27 1.27)) (justify left bottom))
   )
