File: pkg/cnc/boards/voron_v0_toolhead/board-latest/led_buttons.kicad_sch (KiCad schematic)
At the start: 6 parts, among them J11 LED, J12 LED, Q1 BSS138, SW2 USR, U7 SK6812MINI-E

Commit message: Software improvements for the toolhead.
Other:
- note added: "TODO: Switch to a level shifter approach to simplify the software"
Changed lines of the file:
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@@
+    (effects (font (size 1.27 1.27)) (justify left bottom))
+  )
+  (text "TODO: Switch to a level shifter approach to simplify the software"
+    (at 24.13 29.21 0)
     (effects (font (size 1.27 1.27)) (justify left bottom))
   )

Commit message: Flushing some recent changes.
Other:
- note removed: "TODO: Check if this is ok or whether we need to maintain polarity"
Changed lines of the file:
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@@
     (stroke (width 0) (type default))
-  )
-  (text "TODO: Check if this is ok or whether we need to maintain polarity"
-    (at 26.67 24.13 0)
-    (effects (font (size 1.27 1.27)) (justify left bottom))
   )
   (text "TODO: Switch to a level shifter approach to simplify the software"
