File: pkg/cnc/boards/voron_v0_umbilical/board-latest/board-latest.kicad_pcb (KiCad board)
At the start: 2 copper layers, 122 x 37 mm, 3 parts, among them J1 UMB, J3 POWER_IN, J4 USB_IN

Commit message: Flushing some of the recent changes.
Parts:
- moved J1 6.00 mm to (156.8, 115.0)
- turned J4 to 180 degrees
Routing:
- net D-: track 9.02 -> 15.9 mm
- net D+: track 9.02 -> 15.8 mm
- net +24V: track 15.4 -> 21.4 mm
Changed lines of the file:
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@@
   (net 4 "D-")
   (footprint "Components:XT30-2+2_Vertical" (layer "F.Cu")
-    (at 156.75 109)
+    (at 156.75 115)
     (property "Sheetfile" "board-latest.kicad_sch")
     (property "Sheetname" "")
@@
   )
   (footprint "Connector_JST:JST_PH_B3B-PH-SM4-TB_1x03-1MP_P2.00mm_Vertical" (layer "B.Cu")
-    (at 174.53 106.57 90)
+    (at 174.53 106.57 180)
     (descr "JST PH series connector, B3B-PH-SM4-TB (http://www.jst-mfg.com/product/pdf/eng/ePH.pdf), generated with kicad-footprint-generator")
     (tags "connector JST PH vertical")
@@
     (property "ki_keywords" "connector")
     (attr smd)
-    (fp_text reference "J4" (at 0 5.45 90) (layer "B.SilkS")
-        (effects (font (size 1 1) (thickness 0.15)) (justify mirror))
-    )
-    (fp_text value "USB_IN" (at 0 -4.45 90) (layer "B.Fab")
-        (effects (font (size 1 1) (thickness 0.15)) (justify mirror))
-    )
-    (fp_text user "${REFERENCE}" (at 0 1 90) (layer "B.Fab")
+    (fp_text reference "J4" (at 0 5.45) (layer "B.SilkS")
+        (effects (font (size 1 1) (thickness 0.15)) (justify mirror))
+    )
+    (fp_text value "USB_IN" (at 0 -4.45) (layer "B.Fab")
+        (effects (font (size 1 1) (thickness 0.15)) (justify mirror))
+    )
+    (fp_text user "${REFERENCE}" (at 0 1) (layer "B.Fab")
         (effects (font (size 1 1) (thickness 0.15)) (justify mirror))
     )
@@
     (fp_line (start 4.975 -0.75) (end 4.975 4.25)
       (stroke (width 0.1) (type solid)) (layer "B.Fab"))
-    (pad "1" smd roundrect (at -2 -0.5 90) (size 1 5.5) (layers "B.Cu" "B.Paste" "B.Mask") (roundrect_rratio 0.25)
+    (pad "1" smd roundrect (at -2 -0.5 180) (size 1 5.5) (layers "B.Cu" "B.Paste" "B.Mask") (roundrect_rratio 0.25)
       (net 4 "D-") (pinfunction "Pin_1") (pintype "passive"))
-    (pad "2" smd roundrect (at 0 -0.5 90) (size 1 5.5) (layers "B.Cu" "B.Paste" "B.Mask") (roundrect_rratio 0.25)
+    (pad "2" smd roundrect (at 0 -0.5 180) (size 1 5.5) (layers "B.Cu" "B.Paste" "B.Mask") (roundrect_rratio 0.25)
       (net 3 "D+") (pinfunction "Pin_2") (pintype "passive"))
-    (pad "3" smd roundrect (at 2 -0.5 90) (size 1 5.5) (layers "B.Cu" "B.Paste" "B.Mask") (roundrect_rratio 0.25)
+    (pad "3" smd roundrect (at 2 -0.5 180) (size 1 5.5) (layers "B.Cu" "B.Paste" "B.Mask") (roundrect_rratio 0.25)
       (net 2 "GND") (pinfunction "Pin_3") (pintype "passive"))
-    (pad "MP" smd roundrect (at -4.4 1.75 90) (size 1.6 3) (layers "B.Cu" "B.Paste" "B.Mask") (roundrect_rratio 0.15625))
-    (pad "MP" smd roundrect (at 4.4 1.75 90) (size 1.6 3) (layers "B.Cu" "B.Paste" "B.Mask") (roundrect_rratio 0.15625))
+    (pad "MP" smd roundrect (at -4.4 1.75 180) (size 1.6 3) (layers "B.Cu" "B.Paste" "B.Mask") (roundrect_rratio 0.15625))
+    (pad "MP" smd roundrect (at 4.4 1.75 180) (size 1.6 3) (layers "B.Cu" "B.Paste" "B.Mask") (roundrect_rratio 0.15625))
     (model "${KICAD7_3DMODEL_DIR}/Connector_JST.3dshapes/JST_PH_B3B-PH-SM4-TB_1x03-1MP_P2.00mm_Vertical.wrl"
       (offset (xyz 0 0 0))
@@
     (effects (font (size 1.5 1.5) (thickness 0.3) bold) (justify left bottom))
   )
-  (segment (start 153.42 103.87) (end 144.495 103.87) (width 3) (layer "B.Cu") (net 1))
-  (segment (start 156.75 109) (end 156.75 107.2) (width 3) (layer "B.Cu") (net 1))
-  (segment (start 156.75 107.2) (end 153.42 103.87) (width 3) (layer "B.Cu") (net 1))
+  (segment (start 153.42 103.87) (end 156.75 107.2) (width 3) (layer "B.Cu") (net 1))
+  (segment (start 156.75 107.2) (end 156.75 115) (width 3) (layer "B.Cu") (net 1))
+  (segment (start 144.495 103.87) (end 153.42 103.87) (width 3) (layer "B.Cu") (net 1))
   (via (at 161 127) (size 12) (drill 10.6) (layers "F.Cu" "B.Cu") (free) (net 2))
-  (segment (start 174.03 106.57) (end 167.03 106.57) (width 0.4) (layer "B.Cu") (net 3))
-  (segment (start 167.03 106.57) (end 165.6 108) (width 0.4) (layer "B.Cu") (net 3))
-  (segment (start 167.03 108.57) (end 165.6 110) (width 0.4) (layer "B.Cu") (net 4))
-  (segment (start 174.03 108.57) (end 167.03 108.57) (width 0.4) (layer "B.Cu") (net 4))
+  (segment (start 173.83 108.355786) (end 174.53 107.655786) (width 0.4) (layer "B.Cu") (net 3))
+  (segment (start 165.6 114) (end 166.1 114.5) (width 0.4) (layer "B.Cu") (net 3))
+  (segment (start 173.83 110.011852) (end 173.83 108.355786) (width 0.4) (layer "B.Cu") (net 3))
+  (segment (start 169.341852 114.5) (end 173.83 110.011852) (width 0.4) (layer "B.Cu") (net 3))
+  (segment (start 174.53 107.655786) (end 174.53 107.07) (width 0.4) (layer "B.Cu") (net 3))
+  (segment (start 174.53 109.311852) (end 174.53 107.07) (width 0.4) (layer "B.Cu") (net 3))
+  (segment (start 166.1 114.5) (end 169.341852 114.5) (width 0.4) (layer "B.Cu") (net 3))
+  (segment (start 166.1 115.5) (end 169.756038 115.5) (width 0.4) (layer "B.Cu") (net 4))
+  (segment (start 174.636038 110.62) (end 175.221852 110.62) (width 0.4) (layer "B.Cu") (net 4))
+  (segment (start 175.83 107.77) (end 176.53 107.07) (width 0.4) (layer "B.Cu") (net 4))
+  (segment (start 165.6 116) (end 166.1 115.5) (width 0.4) (layer "B.Cu") (net 4))
+  (segment (start 175.221852 110.62) (end 175.83 110.011852) (width 0.4) (layer "B.Cu") (net 4))
+  (segment (start 169.756038 115.5) (end 174.636038 110.62) (width 0.4) (layer "B.Cu") (net 4))
+  (segment (start 175.83 110.011852) (end 175.83 107.77) (width 0.4) (layer "B.Cu") (net 4))
   (zone (net 2) (net_name "GND") (layer "F.Cu") (hatch edge 0.5)
     (priority 1)
