File: pkg/cluster/machines/jbod/boards/backplane-tester/backplane-tester.kicad_pcb (KiCad board)
At the start: 2 copper layers, 75 x 50 mm, 35 parts, among them J1 POWER, J2 BOARD_IN, J3 SAS_OUT, J4 POWER_RES1, J5 POWER_RES2, Q1 DMG2302U, Q2 DMG2305_P, Q3 DMG2305_P, Q4 DMG2302U, Q5 DMG2302U, Q6 DMG2302U, Q8 DMG2302U, Q9 DMG2302U, U1 MCP23008-xSO, U2 NRF52840_ITSY_BITSY

Commit message: Flush some changes
Routing:
- net SAS_V1: track 19.5 -> 16.9 mm
- net GND: track 174.9 -> 172.6 mm
- net SAS_GND2: track 70.3 -> 71.9 mm
- net SAS_GND2_SENSE: track 57.7 -> 58.4 mm
- net +5V: track 60.2 -> 60.9 mm
- net SAS_V2_SENSE: track 58.0 -> 58.5 mm
- added copper zone on B.Cu, net GND

Commit message: Flushing some recent changes.
Routing:
- net SAS_V1: track 16.9 -> 19.5 mm
Changed lines of the file:
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@@
   (segment (start 181.655 143.241) (end 185.401 146.987) (width 1.6) (layer "F.Cu") (net 7))
   (segment (start 172.835 143.51) (end 173.104 143.241) (width 1.6) (layer "B.Cu") (net 7))
+  (segment (start 182.785 146.987) (end 182.737 146.939) (width 0.4) (layer "B.Cu") (net 7))
+  (segment (start 185.401 146.987) (end 182.785 146.987) (width 0.4) (layer "B.Cu") (net 7))
   (segment (start 170.275 143.51) (end 172.835 143.51) (width 1.6) (layer "B.Cu") (net 7))
   (segment (start 185.353 146.939) (end 185.401 146.987) (width 0.4) (layer "B.Cu") (net 7))
