File: pkg/cluster/machines/jbod/boards/backplane-tester/backplane-tester.kicad_sch (KiCad schematic)
At the start: 35 parts, among them J1 POWER, J2 BOARD_IN, J3 SAS_OUT, J4 POWER_RES1, J5 POWER_RES2, Q1 DMG2302U, Q2 DMG2305_P, Q3 DMG2305_P, Q4 DMG2302U, Q5 DMG2302U, Q6 DMG2302U, Q8 DMG2302U, Q9 DMG2302U, U1 MCP23008-xSO, U2 NRF52840_ITSY_BITSY

Commit message: Flush some changes
Parts:
- Q1, Q4, Q5, Q6, Q8, Q9: value DMG2302U -> N-CH
- Q2, Q3: value DMG2305_P -> P-CH
Changed lines of the file:
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@@
       (effects (font (size 1.27 1.27)) (justify left))
     )
-    (property "Value" "DMG2302U" (at 151.13 114.3 0)
+    (property "Value" "N-CH" (at 151.13 114.3 0)
       (effects (font (size 1.27 1.27)) (justify left))
     )
@@
       (effects (font (size 1.27 1.27)) (justify left))
     )
-    (property "Value" "DMG2302U" (at 208.28 67.31 0)
+    (property "Value" "N-CH" (at 208.28 67.31 0)
       (effects (font (size 1.27 1.27)) (justify left))
     )
@@
       (effects (font (size 1.27 1.27)) (justify left))
     )
-    (property "Value" "DMG2302U" (at 208.28 148.59 0)
+    (property "Value" "N-CH" (at 208.28 148.59 0)
       (effects (font (size 1.27 1.27)) (justify left))
     )
@@
       (effects (font (size 1.27 1.27)) (justify left))
     )
-    (property "Value" "DMG2302U" (at 151.13 148.59 0)
+    (property "Value" "N-CH" (at 151.13 148.59 0)
       (effects (font (size 1.27 1.27)) (justify left))
     )
@@
       (effects (font (size 1.27 1.27)) (justify left))
     )
-    (property "Value" "DMG2302U" (at 207.01 114.3 0)
+    (property "Value" "N-CH" (at 207.01 114.3 0)
       (effects (font (size 1.27 1.27)) (justify left))
     )
@@
       (effects (font (size 1.27 1.27)) (justify left))
     )
-    (property "Value" "DMG2305_P" (at 264.16 34.29 0)
+    (property "Value" "P-CH" (at 264.16 34.29 0)
       (effects (font (size 1.27 1.27)) (justify left))
     )
@@
       (effects (font (size 1.27 1.27)) (justify left))
     )
-    (property "Value" "DMG2302U" (at 208.28 34.29 0)
+    (property "Value" "N-CH" (at 208.28 34.29 0)
       (effects (font (size 1.27 1.27)) (justify left))
     )
@@
       (effects (font (size 1.27 1.27)) (justify left))
     )
-    (property "Value" "DMG2305_P" (at 262.89 67.31 0)
-      (effects (font (size 1.27 1.27)) (justify left))
-    )
+    (property "Value" "P-CH" (at 262.89 67.31 0)
+      (effects (font (size 1.27 1.27)) (justify left))
+    )

Commit message: Flushing some recent changes.
Connections:
- net SCL: now also R20.1, U1.1 (SCL), U2.15 (D0/P0.25); no longer R19.1, U1.2 (SDA), U2.16 (D1/P0.24)
- net SDA: now also R19.1, U1.2 (SDA), U2.16 (D1/P0.24); no longer R20.1, U1.1 (SCL), U2.15 (D0/P0.25)
Other:
- note added: "GP7 is output only"
- note added: "Internal pull-up on the MCP is 100K (DOES NOT HAVE AN INTERNAL PULL-DOWN)"
- note removed: "Internal pull-up/down on the MCP is 100K"
Changed lines of the file:
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@@
     (fill (type none))
   )
-  (text "Internal pull-up/down on the MCP is 100K" (at 105.41 64.77 0)
+  (text "Internal pull-up on the MCP is 100K\n(DOES NOT HAVE AN INTERNAL PULL-DOWN)"
+    (at 106.68 67.31 0)
     (effects (font (size 1.27 1.27)) (justify left bottom))
   )
@@
     (effects (font (size 1.27 1.27)) (justify left bottom))
   )
+  (text "GP7 is output only" (at 106.68 73.66 0)
+    (effects (font (size 1.27 1.27)) (justify left bottom))
+  )
   (text "Load for Resistance\nMeasurement" (at 175.26 95.25 0)
     (effects (font (size 2.5 2.5)) (justify left bottom))
@@
     )
   )
-  (global_label "SDA" (shape input) (at 90.17 40.64 180) (fields_autoplaced)
-    (effects (font (size 1.27 1.27)) (justify right))
-    (property "Intersheetrefs" "${INTERSHEET_REFS}" (at 83.6167 40.64 0)
-      (effects (font (size 1.27 1.27)) (justify right) hide)
-    )
-  )
-  (global_label "SCL" (shape input) (at 90.17 43.18 180) (fields_autoplaced)
-    (effects (font (size 1.27 1.27)) (justify right))
-    (property "Intersheetrefs" "${INTERSHEET_REFS}" (at 83.6772 43.18 0)
+  (global_label "SCL" (shape input) (at 90.17 40.64 180) (fields_autoplaced)
+    (effects (font (size 1.27 1.27)) (justify right))
+    (property "Intersheetrefs" "${INTERSHEET_REFS}" (at 83.6772 40.64 0)
+      (effects (font (size 1.27 1.27)) (justify right) hide)
+    )
+  )
+  (global_label "SDA" (shape input) (at 90.17 43.18 180) (fields_autoplaced)
+    (effects (font (size 1.27 1.27)) (justify right))
+    (property "Intersheetrefs" "${INTERSHEET_REFS}" (at 83.6167 43.18 0)
       (effects (font (size 1.27 1.27)) (justify right) hide)
     )
@@
     )
   )
-  (global_label "SCL" (shape input) (at 76.2 139.7 0) (fields_autoplaced)
-    (effects (font (size 1.27 1.27)) (justify left))
-    (property "Intersheetrefs" "${INTERSHEET_REFS}" (at 82.6928 139.7 0)
+  (global_label "SDA" (shape input) (at 76.2 139.7 0) (fields_autoplaced)
+    (effects (font (size 1.27 1.27)) (justify left))
+    (property "Intersheetrefs" "${INTERSHEET_REFS}" (at 82.7533 139.7 0)
       (effects (font (size 1.27 1.27)) (justify left) hide)
     )
@@
     )
   )
-  (global_label "SCL" (shape input) (at 24.13 173.99 180) (fields_autoplaced)
-    (effects (font (size 1.27 1.27)) (justify right))
-    (property "Intersheetrefs" "${INTERSHEET_REFS}" (at 17.6372 173.99 0)
+  (global_label "SDA" (shape input) (at 24.13 173.99 180) (fields_autoplaced)
+    (effects (font (size 1.27 1.27)) (justify right))
+    (property "Intersheetrefs" "${INTERSHEET_REFS}" (at 17.5767 173.99 0)
       (effects (font (size 1.27 1.27)) (justify right) hide)
     )
@@
     )
   )
-  (global_label "SDA" (shape input) (at 76.2 142.24 0) (fields_autoplaced)
-    (effects (font (size 1.27 1.27)) (justify left))
-    (property "Intersheetrefs" "${INTERSHEET_REFS}" (at 82.7533 142.24 0)
+  (global_label "SCL" (shape input) (at 76.2 142.24 0) (fields_autoplaced)
+    (effects (font (size 1.27 1.27)) (justify left))
+    (property "Intersheetrefs" "${INTERSHEET_REFS}" (at 82.6928 142.24 0)
       (effects (font (size 1.27 1.27)) (justify left) hide)
     )
@@
     )
   )
-  (global_label "SDA" (shape input) (at 24.13 181.61 180) (fields_autoplaced)
-    (effects (font (size 1.27 1.27)) (justify right))
-    (property "Intersheetrefs" "${INTERSHEET_REFS}" (at 17.5767 181.61 0)
-      (effects (font (size 1.27 1.27)) (justify right) hide)
-    )
+  (global_label "SCL" (shape input) (at 24.13 181.61 180) (fields_autoplaced)
+    (effects (font (size 1.27 1.27)) (justify right))
+    (property "Intersheetrefs" "${INTERSHEET_REFS}" (at 17.6372 181.61 0)
+      (effects (font (size 1.27 1.27)) (justify right) hide)
+    )
