File: pkg/peripherals/boards/tc2030_adapter/board/board.kicad_pcb (KiCad board)
At the start: 2 copper layers, 40 x 40 mm, 4 parts, among them J1 Conn_02x03_Odd_Even, J2 Conn_02x05_Odd_Even, SW1 SW_Push, SW2 SW_Push

Commit message: Flushing some recent changes.
Other:
- net class Default removed
