File: pkg/cluster/machines/jbod/boards/backplane/backplane.kicad_pcb (KiCad board)
At the start: 4 copper layers, 113.1 x 64 mm, 22 parts, among them CN1 HDD, CN2 HDD, CN3 HDD, CN4 HDD, J1 POWER, J2 MINI_SAS_HD

Commit message: Flushing some recent code changes.
Other:
- board text added: "Use this line as the edge for the 3 disk board"
Changed lines of the file:
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@@
     )
   )
+  (gr_line (start 130.6 48) (end 129 48)
+    (stroke (width 0.15) (type default)) (layer "Dwgs.User"))
+  (gr_line (start 129 48) (end 129.8 49.2)
+    (stroke (width 0.15) (type default)) (layer "Dwgs.User"))
+  (gr_line (start 129.8 49.2) (end 129.8 41.8)
+    (stroke (width 0.15) (type default)) (layer "Dwgs.User"))
+  (gr_line (start 129.8 49.2) (end 130.6 48)
+    (stroke (width 0.15) (type default)) (layer "Dwgs.User"))
   (gr_line (start 129.787 50) (end 129.787 114)
     (stroke (width 0.15) (type default)) (layer "Eco2.User"))
@@
     (effects (font (size 1 1) (thickness 0.15)) (justify left bottom))
   )
+  (gr_text "Use this line as the edge\nfor the 3 disk board" (at 122.8 41) (layer "Dwgs.User")
+    (effects (font (size 1 1) (thickness 0.15)) (justify left bottom))
+  )
