File: pkg/vision/mocap/boards/compute/r9/5v_buck.kicad_sch (KiCad schematic)
At the start: 10 parts, among them U3 LM65645RZTR

Commit message: New mocap compute board revisions.
Parts:
- removed C10: 0.1uF 10V, Capacitor_SMD:C_0603_1608Metric, symbol Device:C_Small
- removed C15: 1uF 10V, Capacitor_SMD:C_0603_1608Metric, symbol Device:C_Small
Connections:
- net BUCK_VCC: no longer U3.5 (MODE_SYNC_TEMP)
- net GND: now also U3.5 (MODE_SYNC_TEMP)
Other:
- note removed: "(Optional) Extra 5V high frequency noise filtering. (put closer to the CM5)"
- note removed: "Note: We are using FPWM mode since AUTO mode has very bad ripple at lower power usage (we mainly lose some low power efficiency) (this is basically the difference between O(100mV) to O(10mV) ripple."
