File: pkg/vision/mocap/boards/compute/r9/mcu.kicad_sch (KiCad schematic)
At the start: 8 parts, among them U1 STM32G031G4Ux, Y1 ASTX-H11-24.000MHZ-T

Commit message: New mocap compute board revisions.
Parts:
- removed C9: 0.1uF 6.6V, Capacitor_SMD:C_0603_1608Metric, symbol Device:C_Small
Changed lines of the file:
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@@
 		)
-	)
-	(junction
-		(at 226.06 133.35)
-		(diameter 0)
-		(color 0 0 0 0)
 	)
 	(no_connect
@@
 	(wire
 		(pts
-			(xy 226.06 142.24) (xy 226.06 144.78)
+			(xy 223.52 85.09) (xy 223.52 86.36)
 		)
 		(stroke
@@
 	(wire
 		(pts
-			(xy 223.52 85.09) (xy 223.52 86.36)
+			(xy 233.68 133.35) (xy 238.76 133.35)
 		)
 		(stroke
@@
 	(wire
 		(pts
-			(xy 233.68 133.35) (xy 238.76 133.35)
+			(xy 215.9 133.35) (xy 228.6 133.35)
 		)
 		(stroke
@@
 	(wire
 		(pts
-			(xy 215.9 133.35) (xy 226.06 133.35)
+			(xy 27.94 157.48) (xy 27.94 158.75)
 		)
 		(stroke
@@
 	(wire
 		(pts
-			(xy 27.94 157.48) (xy 27.94 158.75)
+			(xy 208.28 133.35) (xy 210.82 133.35)
 		)
 		(stroke
@@
 	(wire
 		(pts
-			(xy 208.28 133.35) (xy 210.82 133.35)
+			(xy 223.52 78.74) (xy 223.52 80.01)
 		)
 		(stroke
@@
 	(wire
 		(pts
-			(xy 223.52 78.74) (xy 223.52 80.01)
-		)
-		(stroke
-			(width 0)
-			(type default)
-		)
-	)
-	(wire
-		(pts
 			(xy 27.94 163.83) (xy 27.94 165.1)
-		)
-		(stroke
-			(width 0)
-			(type default)
-		)
-	)
-	(wire
-		(pts
-			(xy 226.06 133.35) (xy 226.06 137.16)
-		)
-		(stroke
-			(width 0)
-			(type default)
-		)
-	)
-	(wire
-		(pts
-			(xy 226.06 133.35) (xy 228.6 133.35)
 		)
 		(stroke
@@
 	)
 	(symbol
-		(lib_id "Device:C_Small")
-		(at 226.06 139.7 180)
-		(unit 1)
-		(exclude_from_sim no)
-		(in_bom yes)
-		(on_board yes)
-		(dnp no)
-		(fields_autoplaced yes)
-		(property "Reference" "C9"
-			(at 228.6 138.4235 0)
-			(effects
-				(font
-					(size 1.27 1.27)
-				)
-				(justify right)
-			)
-		)
-		(property "Value" "0.1uF 6.6V"
-			(at 228.6 140.9635 0)
-			(effects
-				(font
-					(size 1.27 1.27)
-				)
-				(justify right)
-			)
-		)
-		(property "Footprint" "Capacitor_SMD:C_0603_1608Metric"
-			(at 226.06 139.7 0)
-			(effects
-				(font
-					(size 1.27 1.27)
-				)
-				(hide yes)
-			)
-		)
-		(property "Datasheet" "~"
-			(at 226.06 139.7 0)
-			(effects
-				(font
-					(size 1.27 1.27)
-				)
-				(hide yes)
-			)
-		)
-		(property "Description" "Unpolarized capacitor, small symbol"
-			(at 226.06 139.7 0)
-			(effects
-				(font
-					(size 1.27 1.27)
-				)
-				(hide yes)
-			)
-		)
-		(pin "2"
-		)
-		(pin "1"
-		)
-		(instances
-			(project "board-latest"
-				(path "/07db8977-6a06-4c60-94f6-b57660c455bf/85922700-6366-4e41-a4bf-c6411d8c7585"
-					(reference "C9")
-					(unit 1)
-				)
-			)
-		)
-	)
-	(symbol
 		(lib_id "power:GND")
 		(at 223.52 86.36 0)
@@
 					(unit 1)
 				)
-			)
-		)
-	)
-	(symbol
-		(lib_id "power:GND")
-		(at 226.06 144.78 0)
-		(unit 1)
-		(exclude_from_sim no)
-		(in_bom yes)
-		(on_board yes)
-		(dnp no)
-		(fields_autoplaced yes)
-		(property "Reference" "#PWR096"
-			(at 226.06 151.13 0)
-			(effects
-				(font
-					(size 1.27 1.27)
-				)
-				(hide yes)
-			)
-		)
-		(property "Value" "GND"
-			(at 226.06 149.86 0)
-			(effects
-				(font
-					(size 1.27 1.27)
-				)
-			)
-		)
-		(property "Footprint" ""
-			(at 226.06 144.78 0)
-			(effects
-				(font
-					(size 1.27 1.27)
-				)
-				(hide yes)
-			)
-		)
-		(property "Datasheet" ""
-			(at 226.06 144.78 0)
-			(effects
-				(font
-					(size 1.27 1.27)
-				)
-				(hide yes)
-			)
-		)
-		(property "Description" "Power symbol creates a global label with name \"GND\" , ground"
-			(at 226.06 144.78 0)
-			(effects
-				(font
-					(size 1.27 1.27)
-				)
-				(hide yes)
-			)
-		)
-		(pin "1"
-		)
-		(instances
-			(project "board-latest"
-				(path "/07db8977-6a06-4c60-94f6-b57660c455bf/85922700-6366-4e41-a4bf-c6411d8c7585"
-					(reference "#PWR096")
-					(unit 1)
-				)
