File: pkg/media/camera/boards/camera_vb5943/latest/inputs.kicad_sch (KiCad schematic)
At the start: 11 parts, among them J1 FH34SRJ-22S-0.5SH_50_, Q1 BSS138, Q2 BSS138

Commit message: Adding a bunch of new PCB prototypes.
Parts:
- removed R13: 10K, Resistor_SMD:R_0402_1005Metric, symbol Device:R_Small
- added R14, R15: 1.5K, Resistor_SMD:R_0402_1005Metric, symbol Device:R_Small
Connections:
- net ENABLE_3V3: now also R14.2
- net GND: now also R15.1
- new net ENABLE_1V8: R14.1, R15.2
Other:
- note added: "Level shifting reset input from 3.3V to 1.8V Also keep disabled while Raspberry Pi is floating"
- note removed: "Keep disabled while Raspberry Pi is floating"
