File: pkg/media/camera/boards/camera_vb5943/latest/power.kicad_sch (KiCad schematic)
At the start: 25 parts, among them U2 ATtiny402-SS, U3 NCP163ASN280T1G, U4 TLV74318PDBVR, U5 TLV75512PDYDR

Commit message: Adding a bunch of new PCB prototypes.
Parts:
- removed C36: 1uF, Capacitor_SMD:C_0603_1608Metric, symbol Device:C_Small
- removed R10, R11, R9: 10K, Resistor_SMD:R_0402_1005Metric, symbol Device:R_Small
- removed R8: 1.5K, Resistor_SMD:R_0402_1005Metric, symbol Device:R_Small
- removed U2: ATtiny402-SS, Package_SO:SOIC-8_3.9x4.9mm_P1.27mm, symbol MCU_Microchip_ATtiny:ATtiny402-SS
- added C50: 10uF, Capacitor_SMD:C_0603_1608Metric, symbol Device:C_Small
Connections:
- net ENABLE_1V2 is gone; now on net DIGITAL_3V3: U5.3 (EN)
- net ENABLE_1V8 is gone; now on net DIGITAL_3V3: U4.3 (EN)
- net ENABLE_2V8 is gone; now on net ANALOG_3V3: U3.3 (EN)
- net +1V8: now also C50.1
- net GND: now also C50.2
Other:
- note added: "1.2V LDO - LOTS OF HEAT - 178mA typical, 290mA peak"
- note added: "1.8V LDO (io voltage) - ~0.6mA peak"
- note added: "2.8V LDO (sensor analog power) - 38.5mA typical, 40mA peak - Must be high PSSR"
- note removed: "* EN is internally pulled down for this specific LDO model. Usage of a different LDO will likely require installing the pulldown resistor."
- note removed: "1.2V LDO - LOTS OF HEAT - 155mA typical, 250mA peak"
- note removed: "1.8V LDO - ~13mA peak"
- note removed: "2.8V LDO (sensor analog power) - 60mA typical, 115mA peak - Must be high PSSR"
- note removed: "MCU for power sequencing"
- note removed: "The MCU can be programmed either with a SOIC clip or via the CSI connector."
