File: pkg/vision/mocap/boards/led/latest/board-latest.kicad_pcb (KiCad board)
At the start: 4 copper layers, 48 x 80 mm, 46 parts, among them J1 Conn_01x02, J4 INPUT, U2 TPS26625DRCR, U3 TPS922054DMTR

Commit message: Adding newer mocap pcb files (mostly)
Parts:
- R6: value 59k (1%); R_fset -> 28k (1%); R_fset
- U3: value TPS922054DMTR -> TPS922055DMTR
Routing:
- net V_LIMITED: track 12.2 -> 5.85 mm, vias 22 -> 26
- net GND_IR_LED_P: track 18.8 -> 16.1 mm, vias 11 -> 10
- net D9_OUT: vias 16 -> 11
- net D8_OUT: vias 16 -> 11
- net D7_OUT: vias 16 -> 11
- net D6_OUT: vias 16 -> 11
- net D5_OUT: vias 16 -> 11
- net D4_OUT: vias 16 -> 11
- net D3_OUT: vias 16 -> 11
- net D2_OUT: vias 16 -> 11
- net D1_OUT: vias 16 -> 11
- net D11_OUT: vias 16 -> 11
- net D10_OUT: vias 16 -> 11
- removed copper zone on In1.Cu, net D10_OUT
- removed copper zone on In2.Cu, net D10_OUT
- removed copper zone on In1.Cu, net D11_OUT
- removed copper zone on In2.Cu, net D11_OUT
- removed copper zone on In1.Cu, net D1_OUT
- removed copper zone on In2.Cu, net D1_OUT
- removed copper zone on In1.Cu, net D2_OUT
- removed copper zone on In2.Cu, net D2_OUT
- removed copper zone on In1.Cu, net D3_OUT
- removed copper zone on In2.Cu, net D3_OUT
- removed copper zone on In1.Cu, net D4_OUT
- removed copper zone on In2.Cu, net D4_OUT
- removed copper zone on In1.Cu, net D5_OUT
- removed copper zone on In2.Cu, net D5_OUT
- removed copper zone on In1.Cu, net D6_OUT
- removed copper zone on In2.Cu, net D6_OUT
- removed copper zone on In1.Cu, net D7_OUT
- removed copper zone on In2.Cu, net D7_OUT
- removed copper zone on In1.Cu, net D8_OUT
- removed copper zone on In2.Cu, net D8_OUT
- removed copper zone on In1.Cu, net D9_OUT
- removed copper zone on In2.Cu, net D9_OUT
- removed copper zone on In1.Cu, net GND_IR_LED_P
- removed copper zone on In2.Cu, net GND_IR_LED_P
Other:
- board text added: "Mocap LED R7"
- board text removed: "Mocap LED R4"
- board text removed: "TODO: Automotive grade caps for everything here since it will get warm"

Commit message: Adding a bunch of new PCB prototypes.
Parts:
- removed C10: 0.1uF; 100V ; soft, Capacitor_SMD:C_0805_2012Metric
- added R8: 150K, Resistor_SMD:R_0603_1608Metric, B.Cu at (131.8, 172.8)
- C4: value 1uF; 10V -> 1uF; 50V; Soft
Changed lines of the file:
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@@
 		(embedded_fonts no)
 	)
-	(footprint "Capacitor_SMD:C_0805_2012Metric"
+	(footprint "Resistor_SMD:R_0603_1608Metric"
 		(layer "B.Cu")
-		(at 117.4 155.9 180)
-		(descr "Capacitor SMD 0805 (2012 Metric), square (rectangular) end terminal, IPC_7351 nominal, (Body size source: IPC-SM-782 page 76, https://www.pcb-3d.com/wordpress/wp-content/uploads/ipc-sm-782a_amendment_1_and_2.pdf, https://docs.google.com/spreadsheets/d/1BsfQQcO9C6DZCsRaXUlFlo91Tg2WpOkGARC1WS5S8t0/edit?usp=sharing), generated with kicad-footprint-generator")
-		(tags "capacitor")
-		(property "Reference" "C10"
-			(at 0 1.68 0)
+		(at 131.75 172.83 180)
+		(descr "Resistor SMD 0603 (1608 Metric), square (rectangular) end terminal, IPC_7351 nominal, (Body size source: IPC-SM-782 page 72, https://www.pcb-3d.com/wordpress/wp-content/uploads/ipc-sm-782a_amendment_1_and_2.pdf), generated with kicad-footprint-generator")
+		(tags "resistor")
+		(property "Reference" "R8"
+			(at 0 1.43 0)
 			(layer "B.SilkS")
 			(hide yes)
@@
 			)
 		)
-		(property "Value" "0.1uF; 100V ; soft"
-			(at 0 -1.68 0)
+		(property "Value" "150K"
+			(at 0 -1.43 0)
 			(layer "B.Fab")
 			(hide yes)
@@
 			)
 		)
-		(property "Description" "Unpolarized capacitor, small symbol"
+		(property "Description" "Resistor, small symbol"
 			(at 0 0 0)
 			(layer "B.Fab")
@@
 			)
 		)
-		(property ki_fp_filters "C_*")
+		(property ki_fp_filters "R_*")
 		(sheetname "/ir_led/")
 		(sheetfile "ir_led.kicad_sch")
-		(attr smd dnp)
+		(attr smd)
 		(fp_line
-			(start -0.261252 0.735)
-			(end 0.261252 0.735)
+			(start -0.237258 0.5225)
+			(end 0.237258 0.5225)
 			(stroke
 				(width 0.12)
@@
 		)
 		(fp_line
-			(start -0.261252 -0.735)
-			(end 0.261252 -0.735)
+			(start -0.237258 -0.5225)
+			(end 0.237258 -0.5225)
 			(stroke
 				(width 0.12)
@@
 		)
 		(fp_line
-			(start 1.7 0.98)
-			(end 1.7 -0.98)
+			(start 1.48 0.73)
+			(end 1.48 -0.73)
 			(stroke
 				(width 0.05)
@@
 		)
 		(fp_line
-			(start 1.7 -0.98)
-			(end -1.7 -0.98)
+			(start 1.48 -0.73)
+			(end -1.48 -0.73)
 			(stroke
 				(width 0.05)
@@
 		)
 		(fp_line
-			(start -1.7 0.98)
-			(end 1.7 0.98)
+			(start -1.48 0.73)
+			(end 1.48 0.73)
 			(stroke
 				(width 0.05)
@@
 		)
 		(fp_line
-			(start -1.7 -0.98)
-			(end -1.7 0.98)
+			(start -1.48 -0.73)
+			(end -1.48 0.73)
 			(stroke
 				(width 0.05)
@@
 		)
 		(fp_line
-			(start 1 0.625)
-			(end 1 -0.625)
+			(start 0.8 0.4125)
+			(end 0.8 -0.4125)
 			(stroke
 				(width 0.1)
@@
 		)
 		(fp_line
-			(start 1 -0.625)
-			(end -1 -0.625)
+			(start 0.8 -0.4125)
+			(end -0.8 -0.4125)
 			(stroke
 				(width 0.1)
@@
 		)
 		(fp_line
-			(start -1 0.625)
-			(end 1 0.625)
+			(start -0.8 0.4125)
+			(end 0.8 0.4125)
 			(stroke
 				(width 0.1)
@@
 		)
 		(fp_line
-			(start -1 -0.625)
-			(end -1 0.625)
+			(start -0.8 -0.4125)
+			(end -0.8 0.4125)
 			(stroke
 				(width 0.1)
@@
 			(effects
 				(font
-					(size 0.5 0.5)
-					(thickness 0.08)
+					(size 0.4 0.4)
+					(thickness 0.06)
 				)
 				(justify mirror)
@@
 		)
 		(pad "1" smd roundrect
-			(at -0.95 0 180)
-			(size 1 1.45)
+			(at -0.825 0 180)
+			(size 0.8 0.95)
 			(layers "B.Cu" "B.Mask" "B.Paste")
 			(roundrect_rratio 0.25)
@@
 		)
 		(pad "2" smd roundrect
-			(at 0.95 0 180)
-			(size 1 1.45)
+			(at 0.825 0 180)
+			(size 0.8 0.95)
 			(layers "B.Cu" "B.Mask" "B.Paste")
 			(roundrect_rratio 0.25)
-			(net 20 "GND_IR_LED_P")
+			(net 13 "GND")
 			(pintype "passive")
 		)
 		(embedded_fonts no)
-		(model "${KICAD6_3DMODEL_DIR}/Capacitor_SMD.3dshapes/C_0805_2012Metric.wrl"
+		(model "${KICAD6_3DMODEL_DIR}/Resistor_SMD.3dshapes/R_0603_1608Metric.wrl"
 			(offset
 				(xyz 0 0 0)
@@
 			)
 		)
-		(property "Value" "1uF; 10V"
+		(property "Value" "1uF; 50V; Soft"
 			(at 0 -1.43 90)
 			(layer "B.Fab")
