File: pkg/vision/mocap/boards/led/latest/ir_led.kicad_sch (KiCad schematic)
At the start: 41 parts, among them J1 Conn_01x02, U3 TPS922054DMTR

Commit message: Adding newer mocap pcb files (mostly)
Parts:
- R6: value 59k (1%); R_fset -> 28k (1%); R_fset
- U3: value TPS922054DMTR -> TPS922055DMTR
Other:
- note added: "FSET configured for 800kHz switching frequency."
- note removed: "FSET configured for 400kHz switching frequency."
Changed lines of the file:
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@@
 		)
 	)
-	(text "FSET configured for 400kHz switching frequency."
+	(text "FSET configured for 800kHz switching frequency."
 		(exclude_from_sim no)
 		(at 78.994 54.356 0)
@@
 			)
 		)
-		(property "Value" "59k (1%); R_fset"
+		(property "Value" "28k (1%); R_fset"
 			(at 126.238 51.816 0)
 			(effects
@@
 			)
 		)
-		(property "Value" "TPS922054DMTR"
+		(property "Value" "TPS922055DMTR"
 			(at 78.74 20.32 0)
 			(effects

Commit message: Adding a bunch of new PCB prototypes.
Parts:
- added R8: 150K, Resistor_SMD:R_0603_1608Metric, symbol Device:R_Small
- C10: now left out of the parts list
- C4: value 1uF; 10V -> 1uF; 50V; Soft
Connections:
- net GND: now also R8.2
- net V_LIMITED: now also R8.1
Other:
- note added: "Capacitor Bleed Try to discharge if unpowered for 1 minute 150K mainly chosen since we also use it on the compute board"
Changed lines of the file:
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@@
 		)
 	)
+	(rectangle
+		(start 165.1 15.24)
+		(end 210.82 68.58)
+		(stroke
+			(width 0)
+			(type dash)
+		)
+		(fill
+			(type none)
+		)
+	)
 	(text "** Keep smaller values close to the LED driver IC"
 		(exclude_from_sim no)
@@
 		)
 	)
+	(text "Capacitor Bleed\n\nTry to discharge if unpowered\nfor 1 minute\n\n150K mainly chosen since we also\nuse it on the compute board"
+		(exclude_from_sim no)
+		(at 167.64 25.4 0)
+		(effects
+			(font
+				(size 1.27 1.27)
+			)
+			(justify left)
+		)
+	)
 	(text "FSET configured for 800kHz switching frequency."
 		(exclude_from_sim no)
@@
 	(wire
 		(pts
+			(xy 190.5 50.8) (xy 190.5 58.42)
+		)
+		(stroke
+			(width 0)
+			(type default)
+		)
+	)
+	(wire
+		(pts
 			(xy 260.35 63.5) (xy 260.35 52.07)
 		)
@@
 	(wire
 		(pts
+			(xy 190.5 38.1) (xy 190.5 45.72)
+		)
+		(stroke
+			(width 0)
+			(type default)
+		)
+	)
+	(wire
+		(pts
 			(xy 243.84 63.5) (xy 233.68 63.5)
 		)
@@
 	(wire
 		(pts
+			(xy 185.42 38.1) (xy 190.5 38.1)
+		)
+		(stroke
+			(width 0)
+			(type default)
+		)
+	)
+	(wire
+		(pts
 			(xy 115.57 171.45) (xy 121.92 171.45)
 		)
@@
 		)
 	)
+	(global_label "V_LIMITED"
+		(shape input)
+		(at 185.42 38.1 180)
+		(fields_autoplaced yes)
+		(effects
+			(font
+				(size 1.27 1.27)
+			)
+			(justify right)
+		)
+		(property "Intersheetrefs" "${INTERSHEET_REFS}"
+			(at 173.3029 38.1 0)
+			(effects
+				(font
+					(size 1.27 1.27)
+				)
+				(justify right)
+				(hide yes)
+			)
+		)
+	)
 	(global_label "IR_LED_FAULT"
 		(shape input)
@@
 			)
 		)
-		(property "Value" "1uF; 10V"
+		(property "Value" "1uF; 50V; Soft"
 			(at 31.7563 31.75 90)
 			(effects
@@
 	(symbol
 		(lib_id "Device:R_Small")
+		(at 190.5 48.26 0)
+		(unit 1)
+		(exclude_from_sim no)
+		(in_bom yes)
+		(on_board yes)
+		(dnp no)
+		(property "Reference" "R8"
+			(at 194.31 47.244 0)
+			(effects
+				(font
+					(size 1.27 1.27)
+				)
+			)
+		)
+		(property "Value" "150K"
+			(at 195.58 49.53 0)
+			(effects
+				(font
+					(size 1.27 1.27)
+				)
+			)
+		)
+		(property "Footprint" "Resistor_SMD:R_0603_1608Metric"
+			(at 190.5 48.26 0)
+			(effects
+				(font
+					(size 1.27 1.27)
+				)
+				(hide yes)
+			)
+		)
+		(property "Datasheet" "~"
+			(at 190.5 48.26 0)
+			(effects
+				(font
+					(size 1.27 1.27)
+				)
+				(hide yes)
+			)
+		)
+		(property "Description" "Resistor, small symbol"
+			(at 190.5 48.26 0)
+			(effects
+				(font
+					(size 1.27 1.27)
+				)
+				(hide yes)
+			)
+		)
+		(pin "1"
+		)
+		(pin "2"
+		)
+		(instances
+			(project "board-latest"
+				(path "/d67f92a0-3cbd-4ffd-b94a-132745dc8102/207e7a44-1eb7-4104-8be0-83f8765f5816"
+					(reference "R8")
+					(unit 1)
+				)
+			)
+		)
+	)
+	(symbol
+		(lib_id "Device:R_Small")
 		(at 90.17 106.68 270)
 		(unit 1)
@@
 		(unit 1)
 		(exclude_from_sim no)
-		(in_bom yes)
-		(on_board yes)
+		(in_bom no)
+		(on_board no)
 		(dnp yes)
 		(fields_autoplaced yes)
@@
 					(unit 1)
 				)
+			)
+		)
+	)
+	(symbol
+		(lib_id "power:GND")
+		(at 190.5 58.42 0)
+		(unit 1)
+		(exclude_from_sim no)
+		(in_bom yes)
+		(on_board yes)
+		(dnp no)
+		(fields_autoplaced yes)
+		(property "Reference" "#PWR06"
+			(at 190.5 64.77 0)
+			(effects
+				(font
+					(size 1.27 1.27)
+				)
+				(hide yes)
+			)
+		)
+		(property "Value" "GND"
+			(at 190.5 63.5 0)
+			(effects
+				(font
+					(size 1.27 1.27)
+				)
+			)
+		)
+		(property "Footprint" ""
+			(at 190.5 58.42 0)
+			(effects
+				(font
+					(size 1.27 1.27)
+				)
+				(hide yes)
+			)
+		)
+		(property "Datasheet" ""
+			(at 190.5 58.42 0)
+			(effects
+				(font
+					(size 1.27 1.27)
+				)
+				(hide yes)
+			)
+		)
+		(property "Description" "Power symbol creates a global label with name \"GND\" , ground"
+			(at 190.5 58.42 0)
+			(effects
+				(font
+					(size 1.27 1.27)
+				)
+				(hide yes)
+			)
+		)
+		(pin "1"
+		)
+		(instances
+			(project "board-latest"
+				(path "/d67f92a0-3cbd-4ffd-b94a-132745dc8102/207e7a44-1eb7-4104-8be0-83f8765f5816"
+					(reference "#PWR06")
+					(unit 1)
+				)
